File: K_Ozols_MultiVib_MD_1/K_Ozols_MultiVib_MD_1/K_Ozols_MultiVib_MD_1.sch (KiCad schematic (older format))
At the start: 10 parts, among them U1 DMC20402

Commit message: Tika izlabota 1. majasdarba kluuda
Connections:
- net at C1.1, R1.2: now also U1.4 (E2); no longer U1.1 (E1)
- net at C2.1, R3.2: now also U1.5 (B2); no longer U1.2 (B1)
- net at C2.2, R4.2: now also U1.6 (C1); no longer U1.3 (C2)
- net at C1.2, R2.2: now also U1.2 (B1); no longer U1.5 (B2)
- new net: BT1.2 (-), U1.1 (E1), U1.3 (C2)
Changed lines of the file:
@@
 LIBS:valves
 LIBS:dmc20402
+LIBS:K_Ozols_MultiVib_MD_1-cache
 EELAYER 25 0
 EELAYER END
@@
 	5550 3100 5550 3300
 Wire Wire Line
-	5550 3600 5550 4750
-Wire Wire Line
 	5550 3750 5600 3750
 Wire Wire Line
-	5950 3600 5950 3750
+	5950 3600 5950 3900
 Wire Wire Line
-	5900 3750 6150 3750
-Wire Wire Line
-	6250 3750 6350 3750
-Wire Wire Line
-	6700 3600 6700 4750
+	6150 3750 6350 3750
 Wire Wire Line
 	6700 3750 6650 3750
+Connection ~ 6250 3750
+Connection ~ 6700 3750
+Connection ~ 5550 3750
+Wire Wire Line
+	4800 3750 4800 4750
+Connection ~ 5950 3750
+Wire Wire Line
+	5950 3750 5900 3750
+Wire Wire Line
+	5550 3600 5550 3950
+Wire Wire Line
+	6250 3600 6250 3750
+Wire Wire Line
+	4800 4750 5950 4750
 Wire Wire Line
 	6150 4750 6150 4850
-Connection ~ 6250 3750
 Wire Wire Line
-	6700 4750 6350 4750
-Connection ~ 6700 3750
+	6150 4850 5700 4850
 Wire Wire Line
-	6600 3900 6600 4850
+	5700 4850 5700 3900
 Wire Wire Line
-	6600 4850 6150 4850
+	5700 3900 5950 3900
 Wire Wire Line
-	5550 4750 5950 4750
-Connection ~ 5550 3750
+	6700 3850 6000 3850
 Wire Wire Line
-	6250 3600 6250 3900
+	6000 3850 6000 4050
 Wire Wire Line
-	6250 3900 6600 3900
+	6000 4050 5950 4050
+Connection ~ 6700 3850
 Wire Wire Line
-	6350 4050 6350 4000
+	6700 3600 6700 3850
 Wire Wire Line
-	6350 4000 4800 4000
+	6350 4750 6350 4900
 Wire Wire Line
-	4800 4000 4800 3750
+	6350 4900 5600 4900
 Wire Wire Line
-	5950 4050 5950 4000
-Connection ~ 5950 4000
+	5600 4900 5600 4750
+Connection ~ 5600 4750
 Wire Wire Line
-	6150 3750 6150 4050
-Connection ~ 5950 3750
+	6150 4050 6150 3750
+Wire Wire Line
+	6350 4050 6350 3950
+Wire Wire Line
+	6350 3950 5550 3950
 $EndSCHEMATC
