File: K_Ozols_MultiVib_MD_1/K_Ozols_MultiVib_MD_1/K_Ozols_MultiVib_MD_1.sch (KiCad schematic (older format))
At the start: 10 parts, among them U1 DMC20402

Commit message: Izlaboju 1. MD kljuudu
Connections:
- net at BT1.2 (-), U1.1 (E1): now also U1.4 (E2); no longer U1.3 (C2)
- net at C1.1, R1.2: now also U1.3 (C2); no longer U1.4 (E2)
Changed lines of the file:
@@
 Wire Wire Line
 	6000 4050 5950 4050
-Connection ~ 6700 3850
 Wire Wire Line
 	6700 3600 6700 3850
 Wire Wire Line
-	6350 4750 6350 4900
-Wire Wire Line
-	6350 4900 5600 4900
-Wire Wire Line
-	5600 4900 5600 4750
-Connection ~ 5600 4750
-Wire Wire Line
 	6150 4050 6150 3750
-Wire Wire Line
-	6350 4050 6350 3950
-Wire Wire Line
-	6350 3950 5550 3950
 Wire Wire Line
 	6650 3750 6700 3750
 Connection ~ 6700 3750
+Wire Wire Line
+	6350 4050 6650 4050
+Wire Wire Line
+	6650 4050 6650 4950
+Wire Wire Line
+	6650 4950 5600 4950
+Wire Wire Line
+	5600 4950 5600 4750
+Connection ~ 5600 4750
+Wire Wire Line
+	6600 4800 6350 4800
+Wire Wire Line
+	6600 3950 6600 4800
+Wire Wire Line
+	5550 3950 6600 3950
+Wire Wire Line
+	6350 4800 6350 4750
 $EndSCHEMATC
