File: Kursa_darbs_Klavs_Ozols/Indicators.sch (KiCad schematic (older format))
At the start: 89 parts, among them U13 LM3915, U14 LM3915, U15 LM3915, U16 LM3915, U17 LM3915, U18 LM3915, U19 LM317_TO3

Commit message: Shiii ir 5. iteraacija manai platei - layouts
Parts:
- C65, C66: footprint Capacitors_THT:CP_Radial_D10.0mm_P5.00mm -> Capacitors_SMD:CP_Elec_10x10.5
- R91, R92, R93, R94, R95, R96: footprint Resistors_THT:R_Axial_DIN0309_L9.0mm_D3.2mm_P5.08mm_Vertical -> Resistors_SMD:R_0805_HandSoldering
- R97: footprint Resistors_THT:R_Axial_DIN0414_L11.9mm_D4.5mm_P20.32mm_Horizontal -> Resistors_SMD:R_0805_HandSoldering
- RV1, RV10, RV11, RV12, RV16, RV2, RV3, RV4, RV5, RV6, RV7, RV8, RV9: footprint Potentiometers:Potentiometer_Trimmer_Vishay_T7YA_Horizontal -> Potentiometers:Potentiometer_Trimmer_Vishay_TS53YJ
Changed lines of the file:
@@
 EESchema Schematic File Version 2
+LIBS:Kursa_darbs_Klavs_Ozols-rescue
 LIBS:power
 LIBS:device
@@
 F 0 "R91" V 2730 2800 50  0000 C CNN
 F 1 "1.2k" V 2650 2800 50  0000 C CNN
-F 2 "Resistors_THT:R_Axial_DIN0309_L9.0mm_D3.2mm_P5.08mm_Vertical" V 2580 2800 50  0001 C CNN
-F 3 "https://eu.mouser.com/datasheet/2/219/MOS-16613.pdf" H 2650 2800 50  0001 C CNN
+F 2 "Resistors_SMD:R_0805_HandSoldering" V 2580 2800 50  0001 C CNN
+F 3 "https://eu.mouser.com/datasheet/2/219/RN73-11994.pdf" H 2650 2800 50  0001 C CNN
 	1    2650 2800
 	1    0    0    -1
@@
 F 0 "C66" H 10075 1950 50  0000 L CNN
 F 1 "10uF" H 10075 1750 50  0000 L CNN
-F 2 "Capacitors_THT:CP_Radial_D10.0mm_P5.00mm" H 10050 1850 50  0001 C CNN
+F 2 "Capacitors_SMD:CP_Elec_10x10.5" H 10050 1850 50  0001 C CNN
 F 3 "https://eu.mouser.com/datasheet/2/293/e-upx-876312.pdf" H 10050 1850 50  0001 C CNN
 	1    10050 1850
@@
 F 0 "C65" H 10075 850 50  0000 L CNN
 F 1 "10 uF" H 10075 650 50  0000 L CNN
-F 2 "Capacitors_THT:CP_Radial_D10.0mm_P5.00mm" H 10050 750 50  0001 C CNN
+F 2 "Capacitors_SMD:CP_Elec_10x10.5" H 10050 750 50  0001 C CNN
 F 3 "https://eu.mouser.com/datasheet/2/293/e-upx-876312.pdf" H 10050 750 50  0001 C CNN
 	1    10050 750
@@
 F 0 "R97" V 10430 950 50  0000 C CNN
 F 1 "240" V 10350 950 50  0000 C CNN
-F 2 "Resistors_THT:R_Axial_DIN0414_L11.9mm_D4.5mm_P20.32mm_Horizontal" V 10280 950 50  0001 C CNN
-F 3 "https://eu.mouser.com/datasheet/2/219/MOS-16613.pdf" H 10350 950 50  0001 C CNN
+F 2 "Resistors_SMD:R_0805_HandSoldering" V 10280 950 50  0001 C CNN
+F 3 "https://eu.mouser.com/datasheet/2/219/RN73-11994.pdf" H 10350 950 50  0001 C CNN
 	1    10350 950
 	0    1    1    0
@@
 F 0 "RV12" V 10575 1250 50  0000 C CNN
 F 1 "4.7k" V 10650 1250 50  0000 C CNN
-F 2 "Potentiometers:Potentiometer_Trimmer_Vishay_T7YA_Horizontal" H 10750 1250 50  0001 C CNN
-F 3 "" H 10750 1250 50  0001 C CNN
+F 2 "Potentiometers:Potentiometer_Trimmer_Vishay_TS53YJ" H 10750 1250 50  0001 C CNN
+F 3 "https://eu.mouser.com/datasheet/2/427/ts53-239982.pdf" H 10750 1250 50  0001 C CNN
 	1    10750 1250
 	0    1    1    0
@@
 F 0 "RV3" V 2825 3050 50  0000 C CNN
 F 1 "10k" V 2900 3050 50  0000 C CNN
-F 2 "Potentiometers:Potentiometer_Trimmer_Vishay_T7YA_Horizontal" H 3000 3050 50  0001 C CNN
-F 3 "https://eu.mouser.com/datasheet/2/427/t7-91033.pdf" H 3000 3050 50  0001 C CNN
+F 2 "Potentiometers:Potentiometer_Trimmer_Vishay_TS53YJ" H 3000 3050 50  0001 C CNN
+F 3 "https://eu.mouser.com/datasheet/2/427/ts53-239982.pdf" H 3000 3050 50  0001 C CNN
 	1    3000 3050
 	0    -1   -1   0
@@
 F 0 "R92" V 2730 5500 50  0000 C CNN
 F 1 "1.2k" V 2650 5500 50  0000 C CNN
-F 2 "Resistors_THT:R_Axial_DIN0309_L9.0mm_D3.2mm_P5.08mm_Vertical" V 2580 5500 50  0001 C CNN
-F 3 "https://eu.mouser.com/datasheet/2/219/MOS-16613.pdf" H 2650 5500 50  0001 C CNN
+F 2 "Resistors_SMD:R_0805_HandSoldering" V 2580 5500 50  0001 C CNN
+F 3 "https://eu.mouser.com/datasheet/2/219/RN73-11994.pdf" H 2650 5500 50  0001 C CNN
 	1    2650 5500
 	1    0    0    -1
@@
 F 0 "RV4" V 2825 5750 50  0000 C CNN
 F 1 "10k" V 2900 5750 50  0000 C CNN
-F 2 "Potentiometers:Potentiometer_Trimmer_Vishay_T7YA_Horizontal" H 3000 5750 50  0001 C CNN
-F 3 "https://eu.mouser.com/datasheet/2/427/t7-91033.pdf" H 3000 5750 50  0001 C CNN
+F 2 "Potentiometers:Potentiometer_Trimmer_Vishay_TS53YJ" H 3000 5750 50  0001 C CNN
+F 3 "https://eu.mouser.com/datasheet/2/427/ts53-239982.pdf" H 3000 5750 50  0001 C CNN
 	1    3000 5750
 	0    -1   -1   0
@@
 F 0 "R93" V 5730 2900 50  0000 C CNN
 F 1 "1.2k" V 5650 2900 50  0000 C CNN
-F 2 "Resistors_THT:R_Axial_DIN0309_L9.0mm_D3.2mm_P5.08mm_Vertical" V 5580 2900 50  0001 C CNN
-F 3 "https://eu.mouser.com/datasheet/2/219/MOS-16613.pdf" H 5650 2900 50  0001 C CNN
+F 2 "Resistors_SMD:R_0805_HandSoldering" V 5580 2900 50  0001 C CNN
+F 3 "https://eu.mouser.com/datasheet/2/219/RN73-11994.pdf" H 5650 2900 50  0001 C CNN
 	1    5650 2900
 	1    0    0    -1
@@
 F 0 "RV6" V 5825 3150 50  0000 C CNN
 F 1 "10k" V 5900 3150 50  0000 C CNN
-F 2 "Potentiometers:Potentiometer_Trimmer_Vishay_T7YA_Horizontal" H 6000 3150 50  0001 C CNN
-F 3 "https://eu.mouser.com/datasheet/2/427/t7-91033.pdf" H 6000 3150 50  0001 C CNN
+F 2 "Potentiometers:Potentiometer_Trimmer_Vishay_TS53YJ" H 6000 3150 50  0001 C CNN
+F 3 "https://eu.mouser.com/datasheet/2/427/ts53-239982.pdf" H 6000 3150 50  0001 C CNN
 	1    6000 3150
 	0    -1   -1   0
@@
 F 0 "R95" V 8730 2950 50  0000 C CNN
 F 1 "1.2k" V 8650 2950 50  0000 C CNN
-F 2 "Resistors_THT:R_Axial_DIN0309_L9.0mm_D3.2mm_P5.08mm_Vertical" V 8580 2950 50  0001 C CNN
-F 3 "https://eu.mouser.com/datasheet/2/219/MOS-16613.pdf" H 8650 2950 50  0001 C CNN
+F 2 "Resistors_SMD:R_0805_HandSoldering" V 8580 2950 50  0001 C CNN
+F 3 "https://eu.mouser.com/datasheet/2/219/RN73-11994.pdf" H 8650 2950 50  0001 C CNN
 	1    8650 2950
 	1    0    0    -1
@@
 F 0 "RV10" V 8825 3200 50  0000 C CNN
 F 1 "10k" V 8900 3200 50  0000 C CNN
-F 2 "Potentiometers:Potentiometer_Trimmer_Vishay_T7YA_Horizontal" H 9000 3200 50  0001 C CNN
-F 3 "https://eu.mouser.com/datasheet/2/427/t7-91033.pdf" H 9000 3200 50  0001 C CNN
+F 2 "Potentiometers:Potentiometer_Trimmer_Vishay_TS53YJ" H 9000 3200 50  0001 C CNN
+F 3 "https://eu.mouser.com/datasheet/2/427/ts53-239982.pdf" H 9000 3200 50  0001 C CNN
 	1    9000 3200
 	0    -1   -1   0
@@
 F 0 "R94" V 5830 5500 50  0000 C CNN
 F 1 "1.2k" V 5750 5500 50  0000 C CNN
-F 2 "Resistors_THT:R_Axial_DIN0309_L9.0mm_D3.2mm_P5.08mm_Vertical" V 5680 5500 50  0001 C CNN
-F 3 "https://eu.mouser.com/datasheet/2/219/MOS-16613.pdf" H 5750 5500 50  0001 C CNN
+F 2 "Resistors_SMD:R_0805_HandSoldering" V 5680 5500 50  0001 C CNN
+F 3 "https://eu.mouser.com/datasheet/2/219/RN73-11994.pdf" H 5750 5500 50  0001 C CNN
 	1    5750 5500
 	1    0    0    -1
@@
 F 0 "RV7" V 5925 5750 50  0000 C CNN
 F 1 "4.7k" V 6000 5750 50  0000 C CNN
-F 2 "Potentiometers:Potentiometer_Trimmer_Vishay_T7YA_Horizontal" H 6100 5750 50  0001 C CNN
-F 3 "https://eu.mouser.com/datasheet/2/427/t7-91033.pdf" H 6100 5750 50  0001 C CNN
+F 2 "Potentiometers:Potentiometer_Trimmer_Vishay_TS53YJ" H 6100 5750 50  0001 C CNN
+F 3 "https://eu.mouser.com/datasheet/2/427/ts53-239982.pdf" H 6100 5750 50  0001 C CNN
 	1    6100 5750
 	0    -1   -1   0
@@
 F 0 "R96" V 8780 5600 50  0000 C CNN
 F 1 "1.2k" V 8700 5600 50  0000 C CNN
-F 2 "Resistors_THT:R_Axial_DIN0309_L9.0mm_D3.2mm_P5.08mm_Vertical" V 8630 5600 50  0001 C CNN
-F 3 "https://eu.mouser.com/datasheet/2/219/MOS-16613.pdf" H 8700 5600 50  0001 C CNN
+F 2 "Resistors_SMD:R_0805_HandSoldering" V 8630 5600 50  0001 C CNN
+F 3 "https://eu.mouser.com/datasheet/2/219/RN73-11994.pdf" H 8700 5600 50  0001 C CNN
 	1    8700 5600
 	1    0    0    -1
@@
 F 0 "RV11" V 8875 5850 50  0000 C CNN
 F 1 "10k" V 8950 5850 50  0000 C CNN
-F 2 "Potentiometers:Potentiometer_Trimmer_Vishay_T7YA_Horizontal" H 9050 5850 50  0001 C CNN
-F 3 "https://eu.mouser.com/datasheet/2/427/t7-91033.pdf" H 9050 5850 50  0001 C CNN
+F 2 "Potentiometers:Potentiometer_Trimmer_Vishay_TS53YJ" H 9050 5850 50  0001 C CNN
+F 3 "https://eu.mouser.com/datasheet/2/427/ts53-239982.pdf" H 9050 5850 50  0001 C CNN
 	1    9050 5850
 	0    -1   -1   0
@@
 F 0 "RV1" V 1925 5750 50  0000 C CNN
 F 1 "10k" V 2000 5750 50  0000 C CNN
-F 2 "Potentiometers:Potentiometer_Trimmer_Vishay_T7YA_Horizontal" H 2100 5750 50  0001 C CNN
-F 3 "https://eu.mouser.com/datasheet/2/427/t7-91033.pdf" H 2100 5750 50  0001 C CNN
+F 2 "Potentiometers:Potentiometer_Trimmer_Vishay_TS53YJ" H 2100 5750 50  0001 C CNN
+F 3 "https://eu.mouser.com/datasheet/2/427/ts53-239982.pdf" H 2100 5750 50  0001 C CNN
 	1    2100 5750
 	-1   0    0    1
@@
 F 0 "RV8" V 7975 5850 50  0000 C CNN
 F 1 "10k" V 8050 5850 50  0000 C CNN
-F 2 "Potentiometers:Potentiometer_Trimmer_Vishay_T7YA_Horizontal" H 8150 5850 50  0001 C CNN
-F 3 "https://eu.mouser.com/datasheet/2/427/t7-91033.pdf" H 8150 5850 50  0001 C CNN
+F 2 "Potentiometers:Potentiometer_Trimmer_Vishay_TS53YJ" H 8150 5850 50  0001 C CNN
+F 3 "https://eu.mouser.com/datasheet/2/427/ts53-239982.pdf" H 8150 5850 50  0001 C CNN
 	1    8150 5850
 	-1   0    0    1
@@
 F 0 "RV9" V 8025 3200 50  0000 C CNN
 F 1 "10k" V 8100 3200 50  0000 C CNN
-F 2 "Potentiometers:Potentiometer_Trimmer_Vishay_T7YA_Horizontal" H 8200 3200 50  0001 C CNN
-F 3 "https://eu.mouser.com/datasheet/2/427/t7-91033.pdf" H 8200 3200 50  0001 C CNN
+F 2 "Potentiometers:Potentiometer_Trimmer_Vishay_TS53YJ" H 8200 3200 50  0001 C CNN
+F 3 "https://eu.mouser.com/datasheet/2/427/ts53-239982.pdf" H 8200 3200 50  0001 C CNN
 	1    8200 3200
 	-1   0    0    1
@@
 F 0 "RV5" V 5025 3150 50  0000 C CNN
 F 1 "10k" V 5100 3150 50  0000 C CNN
-F 2 "Potentiometers:Potentiometer_Trimmer_Vishay_T7YA_Horizontal" H 5200 3150 50  0001 C CNN
-F 3 "https://eu.mouser.com/datasheet/2/427/t7-91033.pdf" H 5200 3150 50  0001 C CNN
+F 2 "Potentiometers:Potentiometer_Trimmer_Vishay_TS53YJ" H 5200 3150 50  0001 C CNN
+F 3 "https://eu.mouser.com/datasheet/2/427/ts53-239982.pdf" H 5200 3150 50  0001 C CNN
 	1    5200 3150
 	-1   0    0    1
@@
 F 0 "RV2" V 2025 3050 50  0000 C CNN
 F 1 "10k" V 2100 3050 50  0000 C CNN
-F 2 "Potentiometers:Potentiometer_Trimmer_Vishay_T7YA_Horizontal" H 2200 3050 50  0001 C CNN
-F 3 "https://eu.mouser.com/datasheet/2/427/t7-91033.pdf" H 2200 3050 50  0001 C CNN
+F 2 "Potentiometers:Potentiometer_Trimmer_Vishay_TS53YJ" H 2200 3050 50  0001 C CNN
+F 3 "https://eu.mouser.com/datasheet/2/427/ts53-239982.pdf" H 2200 3050 50  0001 C CNN
 	1    2200 3050
 	-1   0    0    1
@@
 F 0 "RV16" V 5025 5850 50  0000 C CNN
 F 1 "10k" V 5100 5850 50  0000 C CNN
-F 2 "Potentiometers:Potentiometer_Trimmer_Vishay_T7YA_Horizontal" H 5200 5850 50  0001 C CNN
-F 3 "https://eu.mouser.com/datasheet/2/427/t7-91033.pdf" H 5200 5850 50  0001 C CNN
+F 2 "Potentiometers:Potentiometer_Trimmer_Vishay_TS53YJ" H 5200 5850 50  0001 C CNN
+F 3 "https://eu.mouser.com/datasheet/2/427/ts53-239982.pdf" H 5200 5850 50  0001 C CNN
 	1    5200 5850
 	-1   0    0    1

Commit message: Shis ir mans meeginaajums iztraseet plati ( nepabeigts- vajag paliidziibu)
Parts:
- added J10: Conn_01x01, Measurement_Points:Measurement_Point_Round-TH_Small, symbol Conn_01x01
Connections:
- net Turpinajums/LED_Supply: now also J10.1 (Pin_1)
Changed lines of the file:
@@
 	5300 5550 5050 5550
 Connection ~ 5300 5550
+$Comp
+L Conn_01x01 J10
+U 1 1 5B1D43C0
+P 8850 650
+F 0 "J10" H 9000 650 50  0000 C CNN
+F 1 "Conn_01x01" H 8850 550 50  0000 C CNN
+F 2 "Measurement_Points:Measurement_Point_Round-TH_Small" H 8850 650 50  0001 C CNN
+F 3 "" H 8850 650 50  0001 C CNN
+	1    8850 650
+	-1   0    0    1
+$EndComp
+Wire Wire Line
+	9050 650  9750 650
+Wire Wire Line
+	9750 650  9750 750
+Connection ~ 9750 750
 $EndSCHEMATC
