File: Kursa_darbs_Klavs_Ozols/Rectifier.sch (KiCad schematic (older format))
At the start: 75 parts, among them U10 TL074, U11 TL074, U12 TL074

Commit message: Shii ir 2. iteraacija kursa darbam!
Connections:
- net Audio10Hz-R: now also C51.1, R67.1; no longer C51.2, R67.2
- net Audio10kHz-R: now also C64.1, R90.1; no longer C64.2, R90.2
- net Audio1kHz-R: now also C58.1, R80.1; no longer C58.2, R80.2
- net Audio2.5kHz-R: now also C60.1, R82.1; no longer C60.2, R82.2
- net Audio200Hz-R: now also C53.1, R69.1; no longer C53.2, R69.2
- net Audio25kHz-R: now also C63.1, R89.1; no longer C63.2, R89.2
- net Audio4.5kHz-R: now also C59.1, R81.1; no longer C59.2, R81.2
- net Audio500Hz-R: now also C54.1, R70.1; no longer C54.2, R70.2
- net Audio50Hz-R: now also C52.1; no longer C52.2
- net GND: now also C51.2, C52.2, C53.2, C54.2, C58.2, C59.2, C60.2, C63.2, C64.2, R67.2, R69.2, R70.2, R80.2, R81.2, R82.2, R89.2, R90.2; no longer C51.1, C52.1, C53.1, C54.1, C58.1, C59.1, C60.1, C63.1, C64.1, R67.1, R69.1, R70.1, R80.1, R81.1, R82.1, R89.1, R90.1
