File: Kursa_darbs_Klavs_Ozols/Kursa_darbs_Klavs_Ozols.kicad_pcb (KiCad board)
At the start: 2 copper layers, 279.4 x 134.6 mm, 317 parts, among them J1 Barosana, J2 Audio-Jack-3, U1 TL074, U10 TL074, U11 TL074, U12 TL074, U13 LM3915, U14 LM3915, U15 LM3915, U16 LM3915, U17 LM3915, U18 LM3915, U19 LM317_TO3, U2 L7808, U20 LM3915, U21 LM3915, U22 LM3915, U3 ICL7660SIPAZ, U4 ICL7660SIPAZ, U5 ICL7660SIPAZ, U6 ICL7660SIPAZ, U7 TL074, U8 TL074, U9 TL074

Commit message: Kursa darba plates 4. iteraacija
Parts:
- removed C66: 10uF, Capacitors_THT:CP_Radial_D10.0mm_P5.00mm
- C47, C51, C52, C53, C54, C58, C60, C62, C63, C64: value 1uF -> 1 uF
- moved C63 57.1 mm to (175.3, 113.4)
- moved C60 55.8 mm to (188.0, 114.1)
- moved D11 55.8 mm to (191.9, 135.5)
- moved D18 55.8 mm to (177.8, 153.9)
- moved D19 55.8 mm to (229.6, 172.1)
- moved D20 55.8 mm to (267.2, 172.1)
- moved D21 55.8 mm to (229.6, 164.0)
- moved D22 55.8 mm to (267.2, 164.0)
- moved D23 55.8 mm to (229.6, 155.8)
- moved D24 55.8 mm to (267.2, 155.8)
- moved D25 55.8 mm to (229.6, 147.4)
- moved D28 55.8 mm to (267.2, 139.6)
- moved D29 55.8 mm to (229.6, 131.2)
- moved D30 55.8 mm to (267.2, 131.2)
- moved D31 55.8 mm to (229.6, 123.1)
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Connections:
- U10 pad 4: GND -> /+8V
- U11 pad 11: GND -> /-8V_2
- U11 pad 4: GND -> /+8V
- U12 pad 11: /-8V_2 -> /-8V_3
- U12 pad 4: GND -> /+8V
- U4 pad 8: GND -> /+8V
- U5 pad 8: GND -> /+8V
- U6 pad 8: GND -> /+8V
- U8 pad 4: GND -> /+8V
- U9 pad 4: GND -> /+8V
Routing:
- net /All_Indicators/Turpinajums/LED_Supply: track 0.00 -> 1626.1 mm
- net /25k: track 0.00 -> 683.1 mm
- net /+8V: track 0.00 -> 505.3 mm
- net GND: track 0.00 -> 463.7 mm
- net /Audio: track 0.00 -> 391.5 mm
- net +12V: track 0.00 -> 311.3 mm
- net /4.5kHz - 2.2 nF/Audio4.5kHz: track 0.00 -> 288.8 mm
- net Net-(D51-Pad1): track 0.00 -> 279.8 mm
- net Net-(D19-Pad1): track 0.00 -> 275.4 mm
- net Net-(D49-Pad1): track 0.00 -> 271.9 mm
- net Net-(D47-Pad1): track 0.00 -> 265.1 mm
- net Net-(D45-Pad1): track 0.00 -> 255.1 mm
- net /10k: track 0.00 -> 247.2 mm
- net /All_Rectifiers/Audio25Hz: track 0.00 -> 233.9 mm
- net /10: track 0.00 -> 215.2 mm
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- added copper zone on B.Cu, net +12V
- added copper zone on F.Cu, net GND
Other:
- copper layers 2 -> 4
- net class Jauda added: clearance 0.2, trace_width 0.75, via_dia 0.6, via_drill 0.4
- net class Mazaakais added: clearance 0.2, trace_width 0.2, via_dia 0.6, via_drill 0.4
- net class Videejais added: clearance 0.2, trace_width 0.5, via_dia 0.6, via_drill 0.4
