File: Kursa_darbs_Klavs_Ozols/Kursa_darbs_Klavs_Ozols.kicad_pcb (KiCad board)
At the start: 4 copper layers, 279.4 x 134.6 mm, 316 parts, among them J1 Barosana, J2 Audio-Jack-3, U1 TL074, U10 TL074, U11 TL074, U12 TL074, U13 LM3915, U14 LM3915, U15 LM3915, U16 LM3915, U17 LM3915, U18 LM3915, U19 LM317_TO3, U2 L7808, U20 LM3915, U21 LM3915, U22 LM3915, U3 ICL7660SIPAZ, U4 ICL7660SIPAZ, U5 ICL7660SIPAZ, U6 ICL7660SIPAZ, U7 TL074, U8 TL074, U9 TL074

Commit message: Vai straadaa ?
Routing:
- net (no net): track 0.11 -> 224.8 mm
Changed lines of the file:
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@@
     (thickness 1.6)
     (drawings 4)
-    (tracks 2370)
+    (tracks 2395)
     (zones 0)
     (modules 316)
@@
     (visible_elements 7FFFFFFF)
     (pcbplotparams
-      (layerselection 0x00030_80000001)
+      (layerselection 0x030ff_80000007)
       (usegerberextensions false)
       (excludeedgelayer true)
@@
       (outputformat 1)
       (mirror false)
-      (drillshape 1)
+      (drillshape 0)
       (scaleselection 1)
       (outputdirectory ""))
@@
   (gr_line (start 63.5 180.467) (end 342.9 180.467) (layer Edge.Cuts) (width 0.15))
   (gr_line (start 63.5 45.847) (end 63.5 180.467) (layer Edge.Cuts) (width 0.15))
+  (segment (start 210.450089 112.754011) (end 208.623194 112.754011) (width 0.25) (layer B.Cu) (net 0))
+  (segment (start 208.623194 112.754011) (end 200.152761 121.224444) (width 0.25) (layer B.Cu) (net 0))
+  (segment (start 200.152761 121.224444) (end 191.614065 121.224444) (width 0.25) (layer B.Cu) (net 0))
+  (segment (start 191.614065 121.224444) (end 187.624992 125.213517) (width 0.25) (layer B.Cu) (net 0))
+  (segment (start 214.62601 149.187747) (end 214.62601 122.594746) (width 0.25) (layer B.Cu) (net 0))
+  (segment (start 187.624992 125.213517) (end 187.624992 129.19751) (width 0.25) (layer B.Cu) (net 0))
+  (segment (start 213.568767 150.24499) (end 214.62601 149.187747) (width 0.25) (layer B.Cu) (net 0))
+  (segment (start 187.624992 129.19751) (end 189.982994 131.555512) (width 0.25) (layer B.Cu) (net 0))
+  (segment (start 189.982994 131.555512) (end 189.982994 133.913514) (width 0.25) (layer B.Cu) (net 0))
+  (segment (start 183.515 48.387) (end 183.594271 48.387) (width 0.25) (layer B.Cu) (net 0))
+  (segment (start 189.982994 133.913514) (end 206.31447 150.24499) (width 0.25) (layer B.Cu) (net 0))
+  (segment (start 213.568767 150.24499) (end 214.285001 149.528756) (width 0.25) (layer B.Cu) (net 0))
+  (segment (start 183.594271 48.387) (end 188.617649 53.410378) (width 0.25) (layer B.Cu) (net 0))
+  (segment (start 189.226522 75.236683) (end 189.226522 85.038557) (width 0.25) (layer B.Cu) (net 0))
+  (segment (start 188.617649 53.410378) (end 188.617649 74.62781) (width 0.25) (layer B.Cu) (net 0))
+  (segment (start 188.617649 74.62781) (end 189.226522 75.236683) (width 0.25) (layer B.Cu) (net 0))
+  (segment (start 189.226522 85.038557) (end 188.892111 85.372968) (width 0.25) (layer B.Cu) (net 0))
+  (segment (start 212.540079 114.844001) (end 210.450089 112.754011) (width 0.25) (layer B.Cu) (net 0))
+  (segment (start 188.892111 85.372968) (end 188.892111 113.280967) (width 0.25) (layer B.Cu) (net 0))
+  (segment (start 188.892111 113.280967) (end 189.982994 114.37185) (width 0.25) (layer B.Cu) (net 0))
+  (segment (start 189.982994 114.37185) (end 189.982994 133.913514) (width 0.25) (layer B.Cu) (net 0))
+  (segment (start 206.31447 150.24499) (end 213.568767 150.24499) (width 0.25) (layer B.Cu) (net 0))
+  (segment (start 214.285001 149.528756) (end 214.285001 115.457081) (width 0.25) (layer B.Cu) (net 0))
+  (segment (start 214.285001 115.457081) (end 213.671921 114.844001) (width 0.25) (layer B.Cu) (net 0))
+  (segment (start 213.671921 114.844001) (end 212.540079 114.844001) (width 0.25) (layer B.Cu) (net 0))
   (segment (start 219.329 123.825) (end 219.329 123.933768) (width 0.25) (layer In2.Cu) (net 0))
   (segment (start 100.33 50.673) (end 100.33 65.786) (width 0.5) (layer F.Cu) (net 1))

Commit message: Shiii ir 5. iteraacija manai platei - layouts
Parts:
- added C66: 10uF, Capacitors_SMD:CP_Elec_10x10.5, B.Cu at (133.3, 180.9)
- added J3: Conn_01x01, Mounting_Holes:MountingHole_3.2mm_M3_Pad, F.Cu at (119.7, 189.2)
- added J4: Conn_01x01, Mounting_Holes:MountingHole_3.2mm_M3_Pad, F.Cu at (120.1, 80.7)
- added J5: Conn_01x01, Mounting_Holes:MountingHole_3.2mm_M3_Pad, F.Cu at (290.6, 190.4)
- added J6: Conn_01x01, Mounting_Holes:MountingHole_3.2mm_M3_Pad, F.Cu at (290.4, 120.7)
- added J7: Conn_01x01, Mounting_Holes:MountingHole_3.2mm_M3_Pad, F.Cu at (153.3, 190.0)
- added J8: Conn_01x01, Mounting_Holes:MountingHole_3.2mm_M3_Pad, F.Cu at (153.0, 120.6)
- C1, C15, C16, C17, C18, C19, C2, C20, C21, C22, C23, C24, C25, C26, C27, C28, C29, C3, C30, C31, C32, C33, C34, C35, C36, C37, C38, C39, C4, C40, C41, C42, C43, C44, C45, C46, C47, C48, C49, C50, C51, C52, C53, C54, C55, C56, C57, C58, C59, C60, C61, C62, C63, C64: footprint Capacitors_THT:C_Axial_L5.1mm_D3.1mm_P10.00mm_Horizontal -> Capacitors_SMD:C_0805_HandSoldering; moved to B.Cu
- C10, C7, C8, C9: footprint Capacitors_THT:CP_Radial_D10.0mm_P5.00mm -> Capacitors_SMD:CP_Elec_4x5.8; moved to B.Cu
- C11, C12, C13, C14, C65: footprint Capacitors_THT:CP_Radial_D10.0mm_P5.00mm -> Capacitors_SMD:CP_Elec_10x10.5; moved to B.Cu
- C5, C6: footprint Capacitors_THT:C_Axial_L3.8mm_D2.6mm_P7.50mm_Horizontal -> Capacitors_SMD:C_1210_HandSoldering; moved to B.Cu
- D1, D10, D11, D12, D13, D14, D15, D16, D17, D18, D2, D3, D4, D5, D6, D7, D8, D9: footprint 1N4148:DO35-3 -> 1N4148:DIOMELF3515N; moved to B.Cu
- J1, J2, U13, U14, U15, U16, U17, U18, U19, U2, U20, U21, U22: moved to B.Cu
- R1, R10, R100, R11, R12, R13, R14, R15, R16, R17, R18, R19, R2, R20, R21, R22, R23, R24, R25, R26, R27, R28, R29, R3, R30, R31, R32, R33, R34, R35, R36, R37, R38, R39, R4, R40, R41, R42, R43, R44, R45, R46, R47, R48, R49, R5, R50, R51, R52, R53, R54, R55, R56, R57, R58, R59, R6, R60, R61, R62, R63, R64, R65, R66, R67, R68, R69, R7, R70, R71, R72, R73, R74, R75, R76, R77, R78, R79, R8, R80, R81, R82, R83, R84, R85, R86, R87, R88, R89, R9, R90, R91, R92, R93, R94, R95, R96, R97, R98, R99: footprint Resistors_THT:R_Axial_DIN0309_L9.0mm_D3.2mm_P5.08mm_Vertical -> Resistors_SMD:R_0805_HandSoldering; moved to B.Cu
- RV1, RV10, RV11, RV12, RV13, RV14, RV15, RV16, RV17, RV18, RV19, RV2, RV3, RV4, RV5, RV6, RV7, RV8, RV9: footprint Potentiometers:Potentiometer_Trimmer_Vishay_T7YA_Horizontal -> Potentiometers:Potentiometer_Trimmer_Vishay_TS53YJ; moved to B.Cu
- U1, U10, U11, U12, U7, U8, U9: footprint TL074:DIL14 -> TL074:SO14; moved to B.Cu
- U3, U4, U5, U6: footprint ICL7660SIPAZ:DIP254P762X533-8 -> Housings_SOIC:SOIC-8_3.9x4.9mm_Pitch1.27mm; moved to B.Cu
- moved R41 201.5 mm to (300.5, 90.8), turned to 180 degrees
- moved R38 200.4 mm to (300.5, 80.5), turned to 180 degrees
- moved R40 196.9 mm to (300.5, 87.7), turned to 0 degrees
- moved R37 196.5 mm to (300.5, 83.6), turned to 0 degrees
- moved C38 179.2 mm to (295.4, 90.8), turned to 0 degrees
- moved C37 178.7 mm to (295.4, 87.8), turned to 0 degrees
- moved C35 178.4 mm to (295.4, 83.5), turned to 0 degrees
- moved C36 178.0 mm to (295.4, 80.5), turned to 0 degrees
- moved R42 172.8 mm to (292.0, 89.3)
- moved R39 171.0 mm to (291.9, 82.1)
- moved R29 166.2 mm to (267.3, 87.9)
- moved R25 165.6 mm to (267.3, 83.3)
- moved R26 165.2 mm to (267.3, 80.2), turned to 180 degrees
- moved R28 161.2 mm to (267.3, 90.9), turned to 0 degrees
- moved U9 159.1 mm to (286.6, 86.3)
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Connections:
- C46 pad 1: /All_Rectifiers/Audio25Hz -> /25 kHz - 470 pF/Audio25kHz
- C49 pad 2: /200Hz - 47nF/Audio200Hz -> /500Hz - 22 nF/Audio500Hz
- C50 pad 2: /500Hz - 22 nF/Audio500Hz -> /200Hz - 47nF/Audio200Hz
- C53 pad 1: /200 -> /500
- C54 pad 1: /500 -> /200
- C56 pad 2: /4.5kHz - 2.2 nF/Audio4.5kHz -> /2.5 kHz- 4.7 nF/Audio2.5kHz
- C57 pad 2: /2.5 kHz- 4.7 nF/Audio2.5kHz -> /4.5kHz - 2.2 nF/Audio4.5kHz
- C59 pad 1: /4.5k -> /2.5k
- C60 pad 1: /2.5k -> /4.5k
- C61 pad 2: /All_Rectifiers/Audio25Hz -> /10 kHz - 1 nF/Audio10kHz
- C62 pad 2: /10 kHz - 1 nF/Audio10kHz -> /25 kHz - 470 pF/Audio25kHz
- C63 pad 1: /25k -> /10k
- C64 pad 1: /10k -> /25k
- D3 pad A: Net-(D3-PadA) -> Net-(D2-PadC)
- D6 pad A: Net-(D2-PadC) -> Net-(D6-PadA)
- D7 pad A: Net-(D3-PadC) -> Net-(D4-PadC)
- D8 pad A: Net-(D4-PadC) -> Net-(D6-PadC)
- R20 pad 1: GND -> Net-(R20-Pad1)
- R21 pad 1: Net-(C24-Pad1) -> Net-(C23-Pad1)
- R21 pad 2: Net-(C23-Pad1) -> Net-(C24-Pad1)
- R22 pad 1: Net-(C25-Pad2) -> Net-(C24-Pad1)
- R22 pad 2: Net-(C24-Pad1) -> Net-(C25-Pad2)
- R23 pad 1: GND -> Net-(R20-Pad1)
- R24 pad 1: /500Hz - 22 nF/Audio500Hz -> Net-(C25-Pad1)
- R24 pad 2: Net-(C25-Pad1) -> /500Hz - 22 nF/Audio500Hz
- R27 pad 1: Net-(C28-Pad1) -> Net-(C27-Pad1)
- R27 pad 2: Net-(C27-Pad1) -> Net-(C28-Pad1)
- R30 pad 1: /1kHz -10 nF/Audio1kHz -> Net-(C29-Pad1)
- R30 pad 2: Net-(C29-Pad1) -> /1kHz -10 nF/Audio1kHz
- R51 pad 1: Net-(C44-Pad1) -> Net-(C43-Pad1)
- R51 pad 2: Net-(C43-Pad1) -> Net-(C44-Pad1)
- R54 pad 1: /All_Rectifiers/Audio25Hz -> /25 kHz - 470 pF/Audio25kHz
- R57 pad 1: Net-(D3-PadA) -> Net-(D4-PadA)
- R58 pad 1: Net-(D4-PadA) -> Net-(D6-PadA)
- R60 pad 1: Net-(D6-PadC) -> Net-(D3-PadC)
- R61 pad 2: Net-(D3-PadA) -> Net-(D4-PadA)
- R62 pad 2: Net-(D4-PadA) -> Net-(D6-PadA)
- R64 pad 2: Net-(D6-PadC) -> Net-(D3-PadC)
- R65 pad 1: /200 -> /500
- R66 pad 1: /500 -> /200
- R68 pad 1: GND -> /50
- R68 pad 2: /50 -> GND
- R69 pad 1: /200 -> /500
- R70 pad 1: /500 -> /200
- R78 pad 1: /4.5k -> /2.5k
- R79 pad 1: /2.5k -> /4.5k
- R81 pad 1: /4.5k -> /2.5k
- R82 pad 1: /2.5k -> /4.5k
- R87 pad 1: /25k -> /10k
- R88 pad 1: /10k -> /25k
- R89 pad 1: /25k -> /10k
- R90 pad 1: /10k -> /25k
- U10 pad 7: /All_Rectifiers/Audio25Hz -> /25 kHz - 470 pF/Audio25kHz
- U11 pad 1: Net-(D3-PadC) -> Net-(D4-PadC)
- U11 pad 11: /-8V_2 -> /-8V_3
- U11 pad 2: Net-(D3-PadA) -> Net-(D4-PadA)
- U11 pad 6: Net-(D4-PadA) -> Net-(D6-PadA)
- U11 pad 7: Net-(D4-PadC) -> Net-(D6-PadC)
- U12 pad 11: /-8V_3 -> /-8V_2
- U7 pad 10: GND -> Net-(R20-Pad1)
- U7 pad 12: GND -> Net-(R20-Pad1)
Routing:
- net /All_Indicators/Turpinajums/LED_Supply: track 1626.1 -> 0.00 mm
- net /25k: track 683.1 -> 0.00 mm
- net /+8V: track 505.3 -> 0.00 mm
- net GND: track 463.7 -> 0.00 mm
- net /Audio: track 391.5 -> 0.00 mm
- net +12V: track 311.3 -> 0.00 mm
- net /4.5kHz - 2.2 nF/Audio4.5kHz: track 288.8 -> 0.00 mm
- net Net-(D51-Pad1): track 279.8 -> 0.00 mm
- net Net-(D19-Pad1): track 275.4 -> 0.00 mm
- net Net-(D49-Pad1): track 271.9 -> 0.00 mm
- net Net-(D47-Pad1): track 265.1 -> 0.00 mm
- net Net-(D45-Pad1): track 255.1 -> 0.00 mm
- net /10k: track 247.2 -> 0.00 mm
- net /All_Rectifiers/Audio25Hz: track 233.9 -> 0.00 mm
- net (no net): track 224.8 -> 0.00 mm
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- removed copper zone on B.Cu, net +12V
- removed copper zone on F.Cu, net GND
Other:
- board size 279.4 x 134.6 mm -> 200.1 x 130 mm

Commit message: Shis ir mans meeginaajums iztraseet plati ( nepabeigts- vajag paliidziibu)
Parts:
- added J10: Conn_01x01, Measurement_Points:Measurement_Point_Round-TH_Small, F.Cu at (124.3, 196.2)
- added J11: Conn_01x01, Measurement_Points:Measurement_Point_Round-TH_Small, F.Cu at (141.6, 99.3)
- added J12: Conn_01x01, Measurement_Points:Measurement_Point_Round-TH_Small, F.Cu at (184.3, 99.6)
- added J13: Conn_01x01, Measurement_Points:Measurement_Point_Round-TH_Small, F.Cu at (223.0, 99.0)
- added J14: Conn_01x01, Measurement_Points:Measurement_Point_Round-TH_Small, F.Cu at (244.4, 99.1)
- added J15: Conn_01x01, Measurement_Points:Measurement_Point_Round-TH_Small, F.Cu at (178.8, 96.5)
- added J16: Conn_01x01, Measurement_Points:Measurement_Point_Round-TH_Small, F.Cu at (220.4, 78.2)
- added J17: Conn_01x01, Measurement_Points:Measurement_Point_Round-TH_Small, F.Cu at (285.7, 74.6)
- added J18: Conn_01x01, Measurement_Points:Measurement_Point_Round-TH_Small, F.Cu at (140.7, 92.5)
- added J19: Conn_01x01, Measurement_Points:Measurement_Point_Round-TH_Small, F.Cu at (273.8, 77.5)
- added J20: Conn_01x01, Measurement_Points:Measurement_Point_Round-TH_Small, F.Cu at (283.6, 92.8)
- added J21: Conn_01x01, Measurement_Points:Measurement_Point_Round-TH_Small, F.Cu at (124.5, 98.6)
- added J22: Conn_01x01, Measurement_Points:Measurement_Point_Round-TH_Small, F.Cu at (302.0, 95.2)
- added J23: Conn_01x01, Measurement_Points:Measurement_Point_Round-TH_Small, F.Cu at (222.9, 94.2)
- added J24: Conn_01x01, Measurement_Points:Measurement_Point_Round-TH_Small, F.Cu at (203.5, 106.2)
- added J25: Conn_01x01, Measurement_Points:Measurement_Point_Round-TH_Small, F.Cu at (179.4, 103.6)
- added J26: Conn_01x01, Measurement_Points:Measurement_Point_Round-TH_Small, F.Cu at (202.0, 209.7)
- added J27: Conn_01x01, Measurement_Points:Measurement_Point_Round-TH_Small, F.Cu at (215.1, 209.1)
- added J28: Conn_01x01, Measurement_Points:Measurement_Point_Round-TH_Small, F.Cu at (285.1, 79.6)
- added J29: Conn_01x01, Measurement_Points:Measurement_Point_Round-TH_Small, F.Cu at (137.2, 111.5)
- added J30: Conn_01x01, Measurement_Points:Measurement_Point_Round-TH_Small, F.Cu at (140.3, 90.0)
- added J31: Conn_01x01, Measurement_Points:Measurement_Point_Round-TH_Small, F.Cu at (159.3, 113.2)
- added J32: Conn_01x01, Measurement_Points:Measurement_Point_Round-TH_Small, F.Cu at (206.2, 206.4)
- added J33: Conn_01x01, Measurement_Points:Measurement_Point_Round-TH_Small, F.Cu at (193.8, 216.4)
- added J34: Conn_01x01, Measurement_Points:Measurement_Point_Round-TH_Small, F.Cu at (323.9, 133.0)
- added J35: Conn_01x01, Measurement_Points:Measurement_Point_Round-TH_Small, F.Cu at (272.8, 111.6)
- added J36: Conn_01x01, Measurement_Points:Measurement_Point_Round-TH_Small, F.Cu at (169.9, 113.5)
- added J37: Conn_01x01, Measurement_Points:Measurement_Point_Round-TH_Small, F.Cu at (263.8, 111.3)
- added J9: Conn_01x01, Measurement_Points:Measurement_Point_Round-TH_Small, F.Cu at (136.9, 188.3)
- moved R98 20.0 mm to (273.6, 141.7)
- moved RV13 20.0 mm to (272.6, 136.3)
- moved R100 19.9 mm to (293.6, 141.4)
- moved RV15 19.7 mm to (292.5, 136.3)
- moved RV19 19.4 mm to (292.8, 171.8)
- moved RV17 19.3 mm to (273.4, 171.8)
- moved R49 0.70 mm to (174.2, 103.0)
- moved R50 0.66 mm to (174.0, 99.7)
- moved R52 0.64 mm to (174.2, 106.1)
- moved C64 0.51 mm to (281.1, 107.7)
- moved C66 0.34 mm to (133.3, 181.2)
Connections:
- R20 pad 1: Net-(R20-Pad1) -> GND
- R23 pad 1: Net-(R20-Pad1) -> GND
- U7 pad 10: Net-(R20-Pad1) -> GND
- U7 pad 12: Net-(R20-Pad1) -> GND
Routing:
- net /All_Indicators/Turpinajums/LED_Supply: track 0.00 -> 903.9 mm
- net GND: track 0.00 -> 380.6 mm
- net /+8V: track 0.00 -> 311.7 mm
- net /Audio: track 0.00 -> 302.6 mm
- net /-8V_2: track 0.00 -> 263.9 mm
- net /-8V_1: track 0.00 -> 241.1 mm
- net /25 kHz - 470 pF/Audio25kHz: track 0.00 -> 155.3 mm
- net /10k: track 0.00 -> 85.1 mm
- net /2.5 kHz- 4.7 nF/Audio2.5kHz: track 0.00 -> 80.5 mm
- net /1k: track 0.00 -> 75.9 mm
- net /200: track 0.00 -> 74.5 mm
- net /50Hz - 220 nF/Audio50Hz: track 0.00 -> 73.4 mm
- net /50: track 0.00 -> 69.3 mm
- net /10Hz-100nF/Audio10Hz: track 0.00 -> 69.0 mm
- net /10: track 0.00 -> 67.8 mm
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- added copper zone on F.Cu, net +12V
- added copper zone on B.Cu, net GND

Commit message: Kursa/Prakses darba pabeigtaa plates versija
Parts:
- added J38: Conn_01x01, Measurement_Points:Measurement_Point_Round-TH_Small, F.Cu at (249.9, 82.0)
- added J39: Conn_01x01, Measurement_Points:Measurement_Point_Round-TH_Small, F.Cu at (259.7, 96.2)
- added J40: Conn_01x01, Measurement_Points:Measurement_Point_Round-TH_Small, F.Cu at (240.1, 101.9)
- added J41: Conn_01x01, Measurement_Points:Measurement_Point_Round-TH_Small, F.Cu at (242.7, 108.9)
- added J42: Conn_01x01, Measurement_Points:Measurement_Point_Round-TH_Small, F.Cu at (247.3, 75.1)
- added J43: Conn_01x01, Measurement_Points:Measurement_Point_Round-TH_Small, F.Cu at (272.9, 104.8)
- added J44: Conn_01x01, Measurement_Points:Measurement_Point_Round-TH_Small, F.Cu at (297.1, 92.7)
- added J45: Conn_01x01, Measurement_Points:Measurement_Point_Round-TH_Small, F.Cu at (283.6, 75.2)
- added J46: Conn_01x01, Measurement_Points:Measurement_Point_Round-TH_Small, F.Cu at (269.1, 101.9)
- added J47: Conn_01x01, Measurement_Points:Measurement_Point_Round-TH_Small, F.Cu at (222.1, 99.9)
- added J48: Conn_01x01, Measurement_Points:Measurement_Point_Round-TH_Small, F.Cu at (193.9, 82.8)
- added J49: Conn_01x01, Measurement_Points:Measurement_Point_Round-TH_Small, F.Cu at (226.7, 83.3)
- added J50: Conn_01x01, Measurement_Points:Measurement_Point_Round-TH_Small, F.Cu at (143.8, 114.0)
- added J51: Conn_01x01, Measurement_Points:Measurement_Point_Round-TH_Small, F.Cu at (125.1, 72.9)
- added J52: Conn_01x01, Measurement_Points:Measurement_Point_Round-TH_Small, F.Cu at (150.1, 114.0)
- moved J33 154.3 mm to (133.7, 74.4)
- moved J21 139.3 mm to (262.9, 82.7)
- moved J15 132.2 mm to (309.8, 78.5)
- moved J31 130.0 mm to (289.3, 111.8)
- moved J26 129.4 mm to (179.6, 82.3)
- moved J22 129.2 mm to (173.2, 104.4)
- moved J27 127.8 mm to (212.3, 81.3)
- moved J34 121.8 mm to (204.8, 107.3)
- moved J17 121.1 mm to (164.9, 66.1)
- moved J37 107.8 mm to (156.2, 104.4)
- moved J25 107.6 mm to (286.9, 99.2)
- moved J32 103.9 mm to (231.1, 105.5)
- moved J23 99.6 mm to (123.3, 97.3)
- moved J24 96.6 mm to (297.2, 82.5)
- moved J18 85.5 mm to (226.1, 95.2)
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Connections:
- J11 pad 1: /50 -> /10Hz-100nF/Audio10Hz
- J12 pad 1: /200 -> /10Hz-100nF/Audio10Hz
- J13 pad 1: /1k -> /50Hz - 220 nF/Audio50Hz
- J14 pad 1: /10k -> /50Hz - 220 nF/Audio50Hz
- J18 pad 1: GND -> /200Hz - 47nF/Audio200Hz
- J19 pad 1: GND -> /200Hz - 47nF/Audio200Hz
- J20 pad 1: GND -> /500Hz - 22 nF/Audio500Hz
- J34 pad 1: GND -> /500Hz - 22 nF/Audio500Hz
Routing:
- net GND: track 380.6 -> 76.7 mm
- net /+8V: track 311.7 -> 582.7 mm
- net /-8V: track 8.63 -> 213.7 mm
- net /-8V_3: track 27.4 -> 182.4 mm
- net /-8V_1: track 241.1 -> 324.0 mm
- net /Audio: track 302.6 -> 356.6 mm
- net /-8V_2: track 263.9 -> 215.6 mm
- net /200Hz - 47nF/Audio200Hz: track 5.78 -> 36.7 mm
- net /1k: track 75.9 -> 106.3 mm
- net /2.5 kHz- 4.7 nF/Audio2.5kHz: track 80.5 -> 53.0 mm
- net +12V: track 36.7 -> 11.5 mm
- net /4.5kHz - 2.2 nF/Audio4.5kHz: track 67.8 -> 42.8 mm
- net Net-(C44-Pad1): track 42.4 -> 25.2 mm
- net /All_Indicators/Turpinajums/LED_Supply: track 903.9 -> 921.0 mm
- net /25k: track 57.8 -> 73.2 mm
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Other:
- board size 200.1 x 130 mm -> 215 x 140 mm
