File: Kursa_darbs_Klavs_Ozols/Kursa_darbs_Klavs_Ozols.kicad_pcb (KiCad board)
At the start: 4 copper layers, 215 x 140 mm, 367 parts, among them J1 Barosana, J10 Conn_01x01, J11 Conn_01x01, J12 Conn_01x01, J13 Conn_01x01, J14 Conn_01x01, J15 Conn_01x01, J16 Conn_01x01, J17 Conn_01x01, J18 Conn_01x01, J19 Conn_01x01, J2 Audio-Jack-3, J20 Conn_01x01, J21 Conn_01x01, J22 Conn_01x01, J23 Conn_01x01, J24 Conn_01x01, J25 Conn_01x01, J26 Conn_01x01, J27 Conn_01x01, J28 Conn_01x01, J29 Conn_01x01, J3 Conn_01x01, J30 Conn_01x01, J31 Conn_01x01, J32 Conn_01x01, J33 Conn_01x01, J34 Conn_01x01, J35 Conn_01x01, J36 Conn_01x01, J37 Conn_01x01, J38 Conn_01x01, J39 Conn_01x01, J4 Conn_01x01, J40 Conn_01x01, J41 Conn_01x01, J42 Conn_01x01, J43 Conn_01x01, J44 Conn_01x01, J45 Conn_01x01, J46 Conn_01x01, J47 Conn_01x01, J48 Conn_01x01, J49 Conn_01x01, J5 Conn_01x01, J50 Conn_01x01, J51 Conn_01x01, J52 Conn_01x01, J6 Conn_01x01, J7 Conn_01x01, J8 Conn_01x01, J9 Conn_01x01, U1 TL074, U10 TL074, U11 TL074, U12 TL074, U13 LM3915, U14 LM3915, U15 LM3915, U16 LM3915, U17 LM3915, U18 LM3915, U19 LM317_TO3, U2 L7808, U20 LM3915, U21 LM3915, U22 LM3915, U3 ICL7660SIPAZ, U4 ICL7660SIPAZ, U5 ICL7660SIPAZ, U6 ICL7660SIPAZ, U7 TL074, U8 TL074, U9 TL074

Commit message: 1. Prototipa finaala versija
Parts:
- added J100: Conn_01x01, Measurement_Points:Measurement_Point_Round-TH_Small, F.Cu at (186.7, 82.9)
- added J101: Conn_01x01, Measurement_Points:Measurement_Point_Round-TH_Small, F.Cu at (186.1, 73.8)
- added J102: Conn_01x01, Measurement_Points:Measurement_Point_Round-TH_Small, F.Cu at (232.7, 178.2)
- added J103: Conn_01x01, Measurement_Points:Measurement_Point_Round-TH_Small, F.Cu at (233.5, 131.4)
- added J104: Conn_01x01, Measurement_Points:Measurement_Point_Round-TH_Small, F.Cu at (166.2, 97.0)
- added J105: Conn_01x01, Measurement_Points:Measurement_Point_Round-TH_Small, F.Cu at (167.2, 102.6)
- added J106: Conn_01x01, Measurement_Points:Measurement_Point_Round-TH_Small, F.Cu at (167.0, 117.7)
- added J107: Conn_01x01, Measurement_Points:Measurement_Point_Round-TH_Small, F.Cu at (177.7, 112.0)
- added J108: Conn_01x01, Measurement_Points:Measurement_Point_Round-TH_Small, F.Cu at (140.4, 86.4)
- added J109: Conn_01x01, Measurement_Points:Measurement_Point_Round-TH_Small, F.Cu at (167.4, 88.1)
- added J110: Conn_01x01, Measurement_Points:Measurement_Point_Round-TH_Small, F.Cu at (147.2, 96.3)
- added J111: Conn_01x01, Measurement_Points:Measurement_Point_Round-TH_Small, F.Cu at (131.4, 132.9)
- added J112: Conn_01x01, Measurement_Points:Measurement_Point_Round-TH_Small, F.Cu at (123.4, 124.9)
- added J113: Conn_01x01, Measurement_Points:Measurement_Point_Round-TH_Small, F.Cu at (123.5, 117.1)
- added J114: Conn_01x01, Measurement_Points:Measurement_Point_Round-TH_Small, F.Cu at (123.4, 108.4)
- added J53: Conn_01x01, Measurement_Points:Measurement_Point_Round-TH_Small, F.Cu at (102.7, 115.2)
- added J54: Conn_01x01, Measurement_Points:Measurement_Point_Round-TH_Small, F.Cu at (157.5, 130.8)
- added J55: Conn_01x01, Measurement_Points:Measurement_Point_Round-TH_Small, F.Cu at (154.4, 177.3)
- added J56: Conn_01x01, Measurement_Points:Measurement_Point_Round-TH_Small, F.Cu at (174.4, 131.5)
- added J57: Conn_01x01, Measurement_Points:Measurement_Point_Round-TH_Small, F.Cu at (171.7, 177.5)
- added J58: Conn_01x01, Measurement_Points:Measurement_Point_Round-TH_Small, F.Cu at (191.3, 177.2)
- added J59: Conn_01x01, Measurement_Points:Measurement_Point_Round-TH_Small, F.Cu at (194.2, 131.8)
- added J60: Conn_01x01, Measurement_Points:Measurement_Point_Round-TH_Small, F.Cu at (213.6, 131.9)
- added J61: Conn_01x01, Measurement_Points:Measurement_Point_Round-TH_Small, F.Cu at (211.6, 177.4)
- added J62: Conn_01x01, Measurement_Points:Measurement_Point_Round-TH_Small, F.Cu at (253.2, 132.3)
- added J63: Conn_01x01, Measurement_Points:Measurement_Point_Round-TH_Small, F.Cu at (251.0, 177.6)
- added J64: Conn_01x01, Measurement_Points:Measurement_Point_Round-TH_Small, F.Cu at (272.5, 131.0)
- added J65: Conn_01x01, Measurement_Points:Measurement_Point_Round-TH_Small, F.Cu at (270.1, 177.6)
- added J66: Conn_01x01, Measurement_Points:Measurement_Point_Round-TH_Small, F.Cu at (292.2, 131.2)
- added J67: Conn_01x01, Measurement_Points:Measurement_Point_Round-TH_Small, F.Cu at (289.2, 177.2)
- added J68: Conn_01x01, Measurement_Points:Measurement_Point_Round-TH_Small, F.Cu at (306.0, 70.3)
- added J69: Conn_01x01, Measurement_Points:Measurement_Point_Round-TH_Small, F.Cu at (309.6, 93.2)
- added J70: Conn_01x01, Measurement_Points:Measurement_Point_Round-TH_Small, F.Cu at (310.2, 106.3)
- added J71: Conn_01x01, Measurement_Points:Measurement_Point_Round-TH_Small, F.Cu at (286.9, 109.2)
- added J72: Conn_01x01, Measurement_Points:Measurement_Point_Round-TH_Small, F.Cu at (267.1, 105.1)
- added J73: Conn_01x01, Measurement_Points:Measurement_Point_Round-TH_Small, F.Cu at (266.4, 92.4)
- added J74: Conn_01x01, Measurement_Points:Measurement_Point_Round-TH_Small, F.Cu at (270.7, 82.6)
- added J75: Conn_01x01, Measurement_Points:Measurement_Point_Round-TH_Small, F.Cu at (272.7, 76.1)
- added J76: Conn_01x01, Measurement_Points:Measurement_Point_Round-TH_Small, F.Cu at (290.9, 82.6)
- added J77: Conn_01x01, Measurement_Points:Measurement_Point_Round-TH_Small, F.Cu at (290.4, 72.6)
- added J78: Conn_01x01, Measurement_Points:Measurement_Point_Round-TH_Small, F.Cu at (289.6, 94.6)
- added J79: Conn_01x01, Measurement_Points:Measurement_Point_Round-TH_Small, F.Cu at (274.8, 81.1)
- added J80: Conn_01x01, Measurement_Points:Measurement_Point_Round-TH_Small, F.Cu at (255.6, 93.7)
- added J81: Conn_01x01, Measurement_Points:Measurement_Point_Round-TH_Small, F.Cu at (255.5, 72.6)
- added J82: Conn_01x01, Measurement_Points:Measurement_Point_Round-TH_Small, F.Cu at (255.4, 82.7)
- added J83: Conn_01x01, Measurement_Points:Measurement_Point_Round-TH_Small, F.Cu at (244.3, 106.3)
- added J84: Conn_01x01, Measurement_Points:Measurement_Point_Round-TH_Small, F.Cu at (246.7, 120.0)
- added J85: Conn_01x01, Measurement_Points:Measurement_Point_Round-TH_Small, F.Cu at (223.1, 109.2)
- added J86: Conn_01x01, Measurement_Points:Measurement_Point_Round-TH_Small, F.Cu at (202.4, 107.4)
- added J87: Conn_01x01, Measurement_Points:Measurement_Point_Round-TH_Small, F.Cu at (200.3, 96.1)
- added J88: Conn_01x01, Measurement_Points:Measurement_Point_Round-TH_Small, F.Cu at (196.5, 120.3)
- added J89: Conn_01x01, Measurement_Points:Measurement_Point_Round-TH_Small, F.Cu at (240.5, 92.3)
- added J90: Conn_01x01, Measurement_Points:Measurement_Point_Round-TH_Small, F.Cu at (236.6, 77.0)
- added J91: Conn_01x01, Measurement_Points:Measurement_Point_Round-TH_Small, F.Cu at (240.5, 76.0)
- added J92: Conn_01x01, Measurement_Points:Measurement_Point_Round-TH_Small, F.Cu at (232.5, 83.9)
- added J93: Conn_01x01, Measurement_Points:Measurement_Point_Round-TH_Small, F.Cu at (220.3, 83.3)
- added J94: Conn_01x01, Measurement_Points:Measurement_Point_Round-TH_Small, F.Cu at (220.0, 72.8)
- added J95: Conn_01x01, Measurement_Points:Measurement_Point_Round-TH_Small, F.Cu at (220.2, 94.5)
- added J96: Conn_01x01, Measurement_Points:Measurement_Point_Round-TH_Small, F.Cu at (203.7, 71.8)
- added J97: Conn_01x01, Measurement_Points:Measurement_Point_Round-TH_Small, F.Cu at (205.7, 81.6)
- added J98: Conn_01x01, Measurement_Points:Measurement_Point_Round-TH_Small, F.Cu at (198.2, 92.8)
- added J99: Conn_01x01, Measurement_Points:Measurement_Point_Round-TH_Small, F.Cu at (186.5, 95.8)
- moved C5 70.5 mm to (111.0, 69.7), turned to 270 degrees
- moved U2 60.4 mm to (105.2, 77.7)
- moved C6 51.1 mm to (111.3, 88.5)
- moved U19 15.3 mm to (105.5, 150.6)
- moved J2 15.1 mm to (159.2, 68.9)
- moved J1 14.8 mm to (145.1, 76.5)
- moved R97 9.94 mm to (115.0, 166.8)
- moved J33 9.88 mm to (137.4, 83.5)
- moved RV16 2.82 mm to (212.0, 171.6)
- moved J52 2.72 mm to (149.3, 116.6)
- moved RV17 2.29 mm to (271.2, 171.7)
- moved RV2 2.28 mm to (132.9, 171.7)
- moved RV19 1.77 mm to (291.0, 171.8)
- moved RV15 1.54 mm to (291.0, 136.2)
- moved RV1 1.52 mm to (193.3, 171.8)
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Connections:
- U5 pad 3: Net-(U5-Pad3) -> GND
Routing:
- net GND: track 76.7 -> 1760.8 mm
- net +12V: track 11.5 -> 779.3 mm
- net /+8V: track 582.7 -> 615.6 mm
- net /All_Indicators/Turpinajums/LED_Supply: track 921.0 -> 930.1 mm
- net Net-(R97-Pad1): track 25.7 -> 32.2 mm
- net Net-(C29-Pad1): track 13.2 -> 16.2 mm
- net Net-(C43-Pad1): track 13.3 -> 15.8 mm
- net Net-(C21-Pad1): track 13.8 -> 15.9 mm
- net /10: track 71.0 -> 73.1 mm
- net Net-(C33-Pad1): track 14.0 -> 16.0 mm
- net /-8V_3: track 182.4 -> 184.2 mm
- net Net-(D55-Pad1): track 23.6 -> 22.0 mm
- net Net-(C31-Pad1): track 13.1 -> 14.6 mm
- net Net-(C15-Pad1): track 16.7 -> 18.1 mm
- net Net-(C25-Pad1): track 14.1 -> 15.5 mm
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- added copper zone on F.Cu, net GND
- removed copper zone on F.Cu, net +12V
Other:
- net class Big added: clearance 0.3, trace_width 1, via_dia 0.9, via_drill 0.4
- net class Default: clearance 0.2 -> 0.3
- net class Jauda: clearance 0.2 -> 0.3
- net class Mazaakais: clearance 0.2 -> 0.3
- net class Videejais: clearance 0.2 -> 0.3; via_dia 0.6 -> 0.8
- rule pad_to_mask_clearance: 0.2 -> 0.3
- rule trace_clearance: 0.2 -> 0.3
