File: Kursa_darbs_Klavs_Ozols/Filter5.sch (KiCad schematic (older format))
At the start: 11 parts, among them U8 TL074

Commit message: Shii ir 2. iteraacija kursa darbam!
Connections:
- net Audio1kHz: now also R30.1; no longer R30.2
- net at C28.1, R28.2, U8.1: now also R27.1; no longer R27.2
- net at C27.1, U8.2 (-): now also R27.2; no longer R27.1
- net at C29.1, U8.6 (-): now also R30.2; no longer R30.1
Changed lines of the file:
@@
 F 3 "" H 4500 2850 50  0001 C CNN
 	1    4500 2850
-	1    0    0    -1
+	0    1    1    0
 $EndComp
 $Comp
@@
 F 3 "" H 7200 2750 50  0001 C CNN
 	1    7200 2750
-	1    0    0    -1
+	0    1    1    0
 $EndComp
 $Comp
@@
 	4250 2650 4900 2650
 Wire Wire Line
-	4500 2650 4500 2700
+	4500 2650 4500 2750
 Wire Wire Line
 	4250 3000 5700 3000
@@
 	6950 2550 7600 2550
 Wire Wire Line
-	7200 2550 7200 2600
+	7200 2550 7200 2650
 Wire Wire Line
 	6950 2900 8400 2900
@@
 Audio1kHz
 Connection ~ 8400 2450
+Wire Wire Line
+	4350 2850 4350 2750
+Wire Wire Line
+	4350 2750 4500 2750
+Wire Wire Line
+	4650 2850 4650 2900
+Wire Wire Line
+	4650 2900 4500 2900
+Wire Wire Line
+	4500 2900 4500 3000
+Wire Wire Line
+	7200 2650 7050 2650
+Wire Wire Line
+	7050 2650 7050 2750
+Wire Wire Line
+	7350 2750 7350 2850
+Wire Wire Line
+	7350 2850 7200 2850
+Wire Wire Line
+	7200 2850 7200 2900
 $EndSCHEMATC

Commit message: Shii ir kursa darba 3. iteraacija
Parts:
- C27, C28, C29, C30: footprint (none) -> Capacitors_THT:C_Axial_L5.1mm_D3.1mm_P10.00mm_Horizontal
- R25, R26, R27, R28, R29, R30: footprint (none) -> Resistors_THT:R_Axial_DIN0309_L9.0mm_D3.2mm_P5.08mm_Vertical
- U8: footprint (none) -> TL074:DIL14
Changed lines of the file:
@@
 F 0 "R25" V 3680 2650 50  0000 C CNN
 F 1 "6.8k" V 3600 2650 50  0000 C CNN
-F 2 "" V 3530 2650 50  0001 C CNN
-F 3 "" H 3600 2650 50  0001 C CNN
+F 2 "Resistors_THT:R_Axial_DIN0309_L9.0mm_D3.2mm_P5.08mm_Vertical" V 3530 2650 50  0001 C CNN
+F 3 "https://eu.mouser.com/datasheet/2/219/MOS-16613.pdf" H 3600 2650 50  0001 C CNN
 	1    3600 2650
 	0    1    1    0
@@
 F 0 "R26" V 3900 2400 50  0000 C CNN
 F 1 "5.1k" V 3800 2400 50  0000 C CNN
-F 2 "" V 3730 2400 50  0001 C CNN
-F 3 "" H 3800 2400 50  0001 C CNN
+F 2 "Resistors_THT:R_Axial_DIN0309_L9.0mm_D3.2mm_P5.08mm_Vertical" V 3730 2400 50  0001 C CNN
+F 3 "https://eu.mouser.com/datasheet/2/219/MOS-16613.pdf" H 3800 2400 50  0001 C CNN
 	1    3800 2400
 	1    0    0    -1
@@
 F 0 "C28" H 4125 3100 50  0000 L CNN
 F 1 "10nF" H 4125 2900 50  0000 L CNN
-F 2 "" H 4138 2850 50  0001 C CNN
-F 3 "" H 4100 3000 50  0001 C CNN
+F 2 "Capacitors_THT:C_Axial_L5.1mm_D3.1mm_P10.00mm_Horizontal" H 4138 2850 50  0001 C CNN
+F 3 "https://eu.mouser.com/datasheet/2/212/KEM_C1046_AXIAL_MOLDED_X7R-1145195.pdf" H 4100 3000 50  0001 C CNN
 	1    4100 3000
 	0    1    1    0
@@
 F 0 "C27" H 4125 2750 50  0000 L CNN
 F 1 "10nF" H 4125 2550 50  0000 L CNN
-F 2 "" H 4138 2500 50  0001 C CNN
-F 3 "" H 4100 2650 50  0001 C CNN
+F 2 "Capacitors_THT:C_Axial_L5.1mm_D3.1mm_P10.00mm_Horizontal" H 4138 2500 50  0001 C CNN
+F 3 "https://eu.mouser.com/datasheet/2/212/KEM_C1046_AXIAL_MOLDED_X7R-1145195.pdf" H 4100 2650 50  0001 C CNN
 	1    4100 2650
 	0    1    1    0
@@
 F 0 "R27" V 4600 2850 50  0000 C CNN
 F 1 "62k" V 4500 2850 50  0000 C CNN
-F 2 "" V 4430 2850 50  0001 C CNN
-F 3 "" H 4500 2850 50  0001 C CNN
+F 2 "Resistors_THT:R_Axial_DIN0309_L9.0mm_D3.2mm_P5.08mm_Vertical" V 4430 2850 50  0001 C CNN
+F 3 "https://eu.mouser.com/datasheet/2/219/MOS-16613.pdf" H 4500 2850 50  0001 C CNN
 	1    4500 2850
 	0    1    1    0
@@
 F 0 "U8" H 5200 2750 50  0000 L CNN
 F 1 "TL074" H 5200 2350 50  0000 L CNN
-F 2 "" H 5150 2650 50  0001 C CNN
+F 2 "TL074:DIL14" H 5150 2650 50  0001 C CNN
 F 3 "" H 5250 2750 50  0001 C CNN
 	1    5200 2550
@@
 F 0 "R28" V 6380 2550 50  0000 C CNN
 F 1 "6.8k" V 6300 2550 50  0000 C CNN
-F 2 "" V 6230 2550 50  0001 C CNN
-F 3 "" H 6300 2550 50  0001 C CNN
+F 2 "Resistors_THT:R_Axial_DIN0309_L9.0mm_D3.2mm_P5.08mm_Vertical" V 6230 2550 50  0001 C CNN
+F 3 "https://eu.mouser.com/datasheet/2/219/MOS-16613.pdf" H 6300 2550 50  0001 C CNN
 	1    6300 2550
 	0    1    1    0
@@
 F 0 "R29" V 6600 2300 50  0000 C CNN
 F 1 "5.1k" V 6500 2300 50  0000 C CNN
-F 2 "" V 6430 2300 50  0001 C CNN
-F 3 "" H 6500 2300 50  0001 C CNN
+F 2 "Resistors_THT:R_Axial_DIN0309_L9.0mm_D3.2mm_P5.08mm_Vertical" V 6430 2300 50  0001 C CNN
+F 3 "https://eu.mouser.com/datasheet/2/219/MOS-16613.pdf" H 6500 2300 50  0001 C CNN
 	1    6500 2300
 	1    0    0    -1
@@
 F 0 "C30" H 6825 3000 50  0000 L CNN
 F 1 "10nF" H 6825 2800 50  0000 L CNN
-F 2 "" H 6838 2750 50  0001 C CNN
-F 3 "" H 6800 2900 50  0001 C CNN
+F 2 "Capacitors_THT:C_Axial_L5.1mm_D3.1mm_P10.00mm_Horizontal" H 6838 2750 50  0001 C CNN
+F 3 "https://eu.mouser.com/datasheet/2/212/KEM_C1046_AXIAL_MOLDED_X7R-1145195.pdf" H 6800 2900 50  0001 C CNN
 	1    6800 2900
 	0    1    1    0
@@
 F 0 "C29" H 6825 2650 50  0000 L CNN
 F 1 "10nF" H 6825 2450 50  0000 L CNN
-F 2 "" H 6838 2400 50  0001 C CNN
-F 3 "" H 6800 2550 50  0001 C CNN
+F 2 "Capacitors_THT:C_Axial_L5.1mm_D3.1mm_P10.00mm_Horizontal" H 6838 2400 50  0001 C CNN
+F 3 "https://eu.mouser.com/datasheet/2/212/KEM_C1046_AXIAL_MOLDED_X7R-1145195.pdf" H 6800 2550 50  0001 C CNN
 	1    6800 2550
 	0    1    1    0
@@
 F 0 "R30" V 7300 2750 50  0000 C CNN
 F 1 "62k" V 7200 2750 50  0000 C CNN
-F 2 "" V 7130 2750 50  0001 C CNN
-F 3 "" H 7200 2750 50  0001 C CNN
+F 2 "Resistors_THT:R_Axial_DIN0309_L9.0mm_D3.2mm_P5.08mm_Vertical" V 7130 2750 50  0001 C CNN
+F 3 "https://eu.mouser.com/datasheet/2/219/MOS-16613.pdf" H 7200 2750 50  0001 C CNN
 	1    7200 2750
 	0    1    1    0
@@
 F 0 "U8" H 7900 2650 50  0000 L CNN
 F 1 "TL074" H 7900 2250 50  0000 L CNN
-F 2 "" H 7850 2550 50  0001 C CNN
+F 2 "TL074:DIL14" H 7850 2550 50  0001 C CNN
 F 3 "" H 7950 2650 50  0001 C CNN
 	2    7900 2450

Commit message: Shiii ir 5. iteraacija manai platei - layouts
Parts:
- C27, C28, C29, C30: footprint Capacitors_THT:C_Axial_L5.1mm_D3.1mm_P10.00mm_Horizontal -> Capacitors_SMD:C_0805_HandSoldering
- R25, R26, R27, R28, R29, R30: footprint Resistors_THT:R_Axial_DIN0309_L9.0mm_D3.2mm_P5.08mm_Vertical -> Resistors_SMD:R_0805_HandSoldering
- U8: footprint TL074:DIL14 -> TL074:SO14
Connections:
- net Audio1kHz: now also R30.2; no longer R30.1
- net at C28.1, R28.2, U8.1: now also R27.2; no longer R27.1
- net at C27.1, U8.2 (-): now also R27.1; no longer R27.2
- net at C29.1, U8.6 (-): now also R30.1; no longer R30.2
Other:
- moved on the sheet: C28, C30, R27, R30
Changed lines of the file:
@@
 EESchema Schematic File Version 2
+LIBS:Kursa_darbs_Klavs_Ozols-rescue
 LIBS:power
 LIBS:device
@@
 Text HLabel 3100 1900 0    60   Input ~ 0
 +8V
-Text HLabel 3100 3250 0    60   Input ~ 0
+Text HLabel 3100 3700 0    60   Input ~ 0
 -8V
 Text HLabel 3100 2150 0    60   Input ~ 0
@@
 F 0 "R25" V 3680 2650 50  0000 C CNN
 F 1 "6.8k" V 3600 2650 50  0000 C CNN
-F 2 "Resistors_THT:R_Axial_DIN0309_L9.0mm_D3.2mm_P5.08mm_Vertical" V 3530 2650 50  0001 C CNN
-F 3 "https://eu.mouser.com/datasheet/2/219/MOS-16613.pdf" H 3600 2650 50  0001 C CNN
+F 2 "Resistors_SMD:R_0805_HandSoldering" V 3530 2650 50  0001 C CNN
+F 3 "https://eu.mouser.com/datasheet/2/219/RN73-11994.pdf" H 3600 2650 50  0001 C CNN
 	1    3600 2650
 	0    1    1    0
@@
 F 0 "R26" V 3900 2400 50  0000 C CNN
 F 1 "5.1k" V 3800 2400 50  0000 C CNN
-F 2 "Resistors_THT:R_Axial_DIN0309_L9.0mm_D3.2mm_P5.08mm_Vertical" V 3730 2400 50  0001 C CNN
-F 3 "https://eu.mouser.com/datasheet/2/219/MOS-16613.pdf" H 3800 2400 50  0001 C CNN
+F 2 "Resistors_SMD:R_0805_HandSoldering" V 3730 2400 50  0001 C CNN
+F 3 "https://eu.mouser.com/datasheet/2/219/RN73-11994.pdf" H 3800 2400 50  0001 C CNN
 	1    3800 2400
 	1    0    0    -1
@@
 L C C28
 U 1 1 5B013960
-P 4100 3000
-F 0 "C28" H 4125 3100 50  0000 L CNN
-F 1 "10nF" H 4125 2900 50  0000 L CNN
-F 2 "Capacitors_THT:C_Axial_L5.1mm_D3.1mm_P10.00mm_Horizontal" H 4138 2850 50  0001 C CNN
-F 3 "https://eu.mouser.com/datasheet/2/212/KEM_C1046_AXIAL_MOLDED_X7R-1145195.pdf" H 4100 3000 50  0001 C CNN
-	1    4100 3000
+P 4100 3450
+F 0 "C28" H 4125 3550 50  0000 L CNN
+F 1 "10nF" H 4125 3350 50  0000 L CNN
+F 2 "Capacitors_SMD:C_0805_HandSoldering" H 4138 3300 50  0001 C CNN
+F 3 "https://eu.mouser.com/datasheet/2/427/vjcommercialseries-222796.pdf" H 4100 3450 50  0001 C CNN
+	1    4100 3450
 	0    1    1    0
 $EndComp
@@
 F 0 "C27" H 4125 2750 50  0000 L CNN
 F 1 "10nF" H 4125 2550 50  0000 L CNN
-F 2 "Capacitors_THT:C_Axial_L5.1mm_D3.1mm_P10.00mm_Horizontal" H 4138 2500 50  0001 C CNN
-F 3 "https://eu.mouser.com/datasheet/2/212/KEM_C1046_AXIAL_MOLDED_X7R-1145195.pdf" H 4100 2650 50  0001 C CNN
+F 2 "Capacitors_SMD:C_0805_HandSoldering" H 4138 2500 50  0001 C CNN
+F 3 "https://eu.mouser.com/datasheet/2/427/vjcommercialseries-222796.pdf" H 4100 2650 50  0001 C CNN
 	1    4100 2650
 	0    1    1    0
@@
 L R R27
 U 1 1 5B013C38
-P 4500 2850
-F 0 "R27" V 4600 2850 50  0000 C CNN
-F 1 "62k" V 4500 2850 50  0000 C CNN
-F 2 "Resistors_THT:R_Axial_DIN0309_L9.0mm_D3.2mm_P5.08mm_Vertical" V 4430 2850 50  0001 C CNN
-F 3 "https://eu.mouser.com/datasheet/2/219/MOS-16613.pdf" H 4500 2850 50  0001 C CNN
-	1    4500 2850
-	0    1    1    0
+P 4500 3050
+F 0 "R27" V 4600 3050 50  0000 C CNN
+F 1 "62k" V 4500 3050 50  0000 C CNN
+F 2 "Resistors_SMD:R_0805_HandSoldering" V 4430 3050 50  0001 C CNN
+F 3 "https://eu.mouser.com/datasheet/2/219/RN73-11994.pdf" H 4500 3050 50  0001 C CNN
+	1    4500 3050
+	1    0    0    -1
 $EndComp
 $Comp
@@
 F 0 "U8" H 5200 2750 50  0000 L CNN
 F 1 "TL074" H 5200 2350 50  0000 L CNN
-F 2 "TL074:DIL14" H 5150 2650 50  0001 C CNN
+F 2 "TL074:SO14" H 5150 2650 50  0001 C CNN
 F 3 "" H 5250 2750 50  0001 C CNN
 	1    5200 2550
@@
 F 0 "R28" V 6380 2550 50  0000 C CNN
 F 1 "6.8k" V 6300 2550 50  0000 C CNN
-F 2 "Resistors_THT:R_Axial_DIN0309_L9.0mm_D3.2mm_P5.08mm_Vertical" V 6230 2550 50  0001 C CNN
-F 3 "https://eu.mouser.com/datasheet/2/219/MOS-16613.pdf" H 6300 2550 50  0001 C CNN
+F 2 "Resistors_SMD:R_0805_HandSoldering" V 6230 2550 50  0001 C CNN
+F 3 "https://eu.mouser.com/datasheet/2/219/RN73-11994.pdf" H 6300 2550 50  0001 C CNN
 	1    6300 2550
 	0    1    1    0
@@
 F 0 "R29" V 6600 2300 50  0000 C CNN
 F 1 "5.1k" V 6500 2300 50  0000 C CNN
-F 2 "Resistors_THT:R_Axial_DIN0309_L9.0mm_D3.2mm_P5.08mm_Vertical" V 6430 2300 50  0001 C CNN
-F 3 "https://eu.mouser.com/datasheet/2/219/MOS-16613.pdf" H 6500 2300 50  0001 C CNN
+F 2 "Resistors_SMD:R_0805_HandSoldering" V 6430 2300 50  0001 C CNN
+F 3 "https://eu.mouser.com/datasheet/2/219/RN73-11994.pdf" H 6500 2300 50  0001 C CNN
 	1    6500 2300
 	1    0    0    -1
@@
 L C C30
 U 1 1 5B01451E
-P 6800 2900
-F 0 "C30" H 6825 3000 50  0000 L CNN
-F 1 "10nF" H 6825 2800 50  0000 L CNN
-F 2 "Capacitors_THT:C_Axial_L5.1mm_D3.1mm_P10.00mm_Horizontal" H 6838 2750 50  0001 C CNN
-F 3 "https://eu.mouser.com/datasheet/2/212/KEM_C1046_AXIAL_MOLDED_X7R-1145195.pdf" H 6800 2900 50  0001 C CNN
-	1    6800 2900
+P 6800 3350
+F 0 "C30" H 6825 3450 50  0000 L CNN
+F 1 "10nF" H 6825 3250 50  0000 L CNN
+F 2 "Capacitors_SMD:C_0805_HandSoldering" H 6838 3200 50  0001 C CNN
+F 3 "https://eu.mouser.com/datasheet/2/427/vjcommercialseries-222796.pdf" H 6800 3350 50  0001 C CNN
+	1    6800 3350
 	0    1    1    0
 $EndComp
@@
 F 0 "C29" H 6825 2650 50  0000 L CNN
 F 1 "10nF" H 6825 2450 50  0000 L CNN
-F 2 "Capacitors_THT:C_Axial_L5.1mm_D3.1mm_P10.00mm_Horizontal" H 6838 2400 50  0001 C CNN
-F 3 "https://eu.mouser.com/datasheet/2/212/KEM_C1046_AXIAL_MOLDED_X7R-1145195.pdf" H 6800 2550 50  0001 C CNN
+F 2 "Capacitors_SMD:C_0805_HandSoldering" H 6838 2400 50  0001 C CNN
+F 3 "https://eu.mouser.com/datasheet/2/427/vjcommercialseries-222796.pdf" H 6800 2550 50  0001 C CNN
 	1    6800 2550
 	0    1    1    0
@@
 L R R30
 U 1 1 5B014530
-P 7200 2750
-F 0 "R30" V 7300 2750 50  0000 C CNN
-F 1 "62k" V 7200 2750 50  0000 C CNN
-F 2 "Resistors_THT:R_Axial_DIN0309_L9.0mm_D3.2mm_P5.08mm_Vertical" V 7130 2750 50  0001 C CNN
-F 3 "https://eu.mouser.com/datasheet/2/219/MOS-16613.pdf" H 7200 2750 50  0001 C CNN
-	1    7200 2750
-	0    1    1    0
+P 7200 2950
+F 0 "R30" V 7300 2950 50  0000 C CNN
+F 1 "62k" V 7200 2950 50  0000 C CNN
+F 2 "Resistors_SMD:R_0805_HandSoldering" V 7130 2950 50  0001 C CNN
+F 3 "https://eu.mouser.com/datasheet/2/219/RN73-11994.pdf" H 7200 2950 50  0001 C CNN
+	1    7200 2950
+	1    0    0    -1
 $EndComp
 $Comp
@@
 F 0 "U8" H 7900 2650 50  0000 L CNN
 F 1 "TL074" H 7900 2250 50  0000 L CNN
-F 2 "TL074:DIL14" H 7850 2550 50  0001 C CNN
+F 2 "TL074:SO14" H 7850 2550 50  0001 C CNN
 F 3 "" H 7950 2650 50  0001 C CNN
 	2    7900 2450
 	1    0    0    -1
 $EndComp
+Text HLabel 8900 2450 2    60   Output ~ 0
+Audio1kHz
 Wire Wire Line
 	3750 2650 3950 2650
 Wire Wire Line
-	3800 2550 3800 3000
+	3800 2550 3800 3450
 Connection ~ 3800 2650
 Wire Wire Line
@@
 	3400 2200 4900 2200
 Wire Wire Line
-	3800 3000 3950 3000
+	3800 3450 3950 3450
 Wire Wire Line
 	4250 2650 4900 2650
 Wire Wire Line
-	4500 2650 4500 2750
-Wire Wire Line
-	4250 3000 5700 3000
-Wire Wire Line
-	4900 2050 4900 2450
+	5700 3450 4250 3450
 Connection ~ 3800 2200
-Connection ~ 4500 2650
-Wire Wire Line
-	5100 3250 5100 2850
-Wire Wire Line
-	3100 3250 5100 3250
-Wire Wire Line
-	5100 1800 5100 2250
-Wire Wire Line
-	3100 1900 5100 1900
-Wire Wire Line
-	5700 3000 5700 2550
-Connection ~ 4500 3000
+Wire Wire Line
+	5100 2850 5100 3700
+Wire Wire Line
+	7800 3700 3100 3700
+Wire Wire Line
+	3100 1900 7800 1900
+Wire Wire Line
+	5700 2550 5700 3450
+Connection ~ 4500 3450
 Wire Wire Line
 	3450 2650 3150 2650
@@
 	6450 2550 6650 2550
 Wire Wire Line
-	6500 2450 6500 2900
+	6500 2450 6500 3350
 Connection ~ 6500 2550
 Wire Wire Line
 	6500 2100 6500 2150
 Wire Wire Line
-	6100 2100 7600 2100
-Wire Wire Line
-	6500 2900 6650 2900
+	4900 2100 7600 2100
 Wire Wire Line
 	6950 2550 7600 2550
-Wire Wire Line
-	7200 2550 7200 2650
-Wire Wire Line
-	6950 2900 8400 2900
 Wire Wire Line
 	7600 2100 7600 2350
@@
 Connection ~ 7200 2550
 Wire Wire Line
-	7800 3150 7800 2750
-Wire Wire Line
-	5100 3150 7800 3150
-Wire Wire Line
-	7800 1800 7800 2150
-Wire Wire Line
-	5100 1800 7800 1800
-Wire Wire Line
-	8400 2900 8400 2450
-Connection ~ 7200 2900
-Wire Wire Line
-	6100 2050 6100 2100
-Wire Wire Line
-	4900 2050 6100 2050
+	7800 2750 7800 3700
+Wire Wire Line
+	8400 3350 8400 2450
 Wire Wire Line
 	8200 2450 8900 2450
@@
 Connection ~ 5100 1900
 Connection ~ 4900 2200
-Connection ~ 5100 3150
-Text HLabel 8900 2450 2    60   Output ~ 0
-Audio1kHz
 Connection ~ 8400 2450
 Wire Wire Line
-	4350 2850 4350 2750
-Wire Wire Line
-	4350 2750 4500 2750
-Wire Wire Line
-	4650 2850 4650 2900
-Wire Wire Line
-	4650 2900 4500 2900
-Wire Wire Line
-	4500 2900 4500 3000
-Wire Wire Line
-	7200 2650 7050 2650
-Wire Wire Line
-	7050 2650 7050 2750
-Wire Wire Line
-	7350 2750 7350 2850
-Wire Wire Line
-	7350 2850 7200 2850
-Wire Wire Line
-	7200 2850 7200 2900
+	4500 3200 4500 3450
+Wire Wire Line
+	4500 2900 4500 2650
+Connection ~ 4500 2650
+Wire Wire Line
+	6500 3350 6650 3350
+Wire Wire Line
+	6950 3350 8400 3350
+Wire Wire Line
+	7200 3350 7200 3100
+Wire Wire Line
+	7200 2800 7200 2550
+Connection ~ 7200 3350
+Wire Wire Line
+	4900 2100 4900 2450
+Wire Wire Line
+	5100 1900 5100 2250
+Wire Wire Line
+	7800 1900 7800 2150
+Connection ~ 5100 3700
 $EndSCHEMATC
