File: Kursa_darbs_Klavs_Ozols/Filter6.sch (KiCad schematic (older format))
At the start: 11 parts, among them U8 TL074

Commit message: Shii ir kursa darba 3. iteraacija
Parts:
- C31, C32, C33, C34: footprint (none) -> Capacitors_THT:C_Axial_L5.1mm_D3.1mm_P10.00mm_Horizontal
- R31, R32, R33, R34, R35, R36: footprint (none) -> Resistors_THT:R_Axial_DIN0309_L9.0mm_D3.2mm_P5.08mm_Vertical
- U8: footprint (none) -> TL074:DIL14
Changed lines of the file:
@@
 F 0 "U8" H 3850 3300 50  0000 L CNN
 F 1 "TL074" H 3850 2900 50  0000 L CNN
-F 2 "" H 3800 3200 50  0001 C CNN
+F 2 "TL074:DIL14" H 3800 3200 50  0001 C CNN
 F 3 "" H 3900 3300 50  0001 C CNN
 	3    3850 3100
@@
 F 0 "R31" V 2430 3200 50  0000 C CNN
 F 1 "6.8k" V 2350 3200 50  0000 C CNN
-F 2 "" V 2280 3200 50  0001 C CNN
-F 3 "" H 2350 3200 50  0001 C CNN
+F 2 "Resistors_THT:R_Axial_DIN0309_L9.0mm_D3.2mm_P5.08mm_Vertical" V 2280 3200 50  0001 C CNN
+F 3 "https://eu.mouser.com/datasheet/2/219/MOS-16613.pdf" H 2350 3200 50  0001 C CNN
 	1    2350 3200
 	0    1    1    0
@@
 F 0 "R32" V 2680 3000 50  0000 C CNN
 F 1 "5.1k" V 2600 3000 50  0000 C CNN
-F 2 "" V 2530 3000 50  0001 C CNN
-F 3 "" H 2600 3000 50  0001 C CNN
+F 2 "Resistors_THT:R_Axial_DIN0309_L9.0mm_D3.2mm_P5.08mm_Vertical" V 2530 3000 50  0001 C CNN
+F 3 "https://eu.mouser.com/datasheet/2/219/MOS-16613.pdf" H 2600 3000 50  0001 C CNN
 	1    2600 3000
 	1    0    0    -1
@@
 F 0 "C31" H 3075 3300 50  0000 L CNN
 F 1 "4.7 nF" H 3075 3100 50  0000 L CNN
-F 2 "" H 3088 3050 50  0001 C CNN
-F 3 "" H 3050 3200 50  0001 C CNN
+F 2 "Capacitors_THT:C_Axial_L5.1mm_D3.1mm_P10.00mm_Horizontal" H 3088 3050 50  0001 C CNN
+F 3 "https://eu.mouser.com/datasheet/2/212/KEM_C1046_AXIAL_MOLDED_X7R-1145195.pdf" H 3050 3200 50  0001 C CNN
 	1    3050 3200
 	0    1    1    0
@@
 F 0 "C32" H 3075 3700 50  0000 L CNN
 F 1 "4.7 nF" H 3075 3500 50  0000 L CNN
-F 2 "" H 3088 3450 50  0001 C CNN
-F 3 "" H 3050 3600 50  0001 C CNN
+F 2 "Capacitors_THT:C_Axial_L5.1mm_D3.1mm_P10.00mm_Horizontal" H 3088 3450 50  0001 C CNN
+F 3 "https://eu.mouser.com/datasheet/2/212/KEM_C1046_AXIAL_MOLDED_X7R-1145195.pdf" H 3050 3600 50  0001 C CNN
 	1    3050 3600
 	0    1    1    0
@@
 F 0 "R33" V 3480 3400 50  0000 C CNN
 F 1 "62k" V 3400 3400 50  0000 C CNN
-F 2 "" V 3330 3400 50  0001 C CNN
-F 3 "" H 3400 3400 50  0001 C CNN
+F 2 "Resistors_THT:R_Axial_DIN0309_L9.0mm_D3.2mm_P5.08mm_Vertical" V 3330 3400 50  0001 C CNN
+F 3 "https://eu.mouser.com/datasheet/2/219/MOS-16613.pdf" H 3400 3400 50  0001 C CNN
 	1    3400 3400
 	1    0    0    -1
@@
 F 0 "R34" V 4730 3100 50  0000 C CNN
 F 1 "6.8k" V 4650 3100 50  0000 C CNN
-F 2 "" V 4580 3100 50  0001 C CNN
-F 3 "" H 4650 3100 50  0001 C CNN
+F 2 "Resistors_THT:R_Axial_DIN0309_L9.0mm_D3.2mm_P5.08mm_Vertical" V 4580 3100 50  0001 C CNN
+F 3 "https://eu.mouser.com/datasheet/2/219/MOS-16613.pdf" H 4650 3100 50  0001 C CNN
 	1    4650 3100
 	0    1    1    0
@@
 F 0 "R35" V 4980 2900 50  0000 C CNN
 F 1 "5.1k" V 4900 2900 50  0000 C CNN
-F 2 "" V 4830 2900 50  0001 C CNN
-F 3 "" H 4900 2900 50  0001 C CNN
+F 2 "Resistors_THT:R_Axial_DIN0309_L9.0mm_D3.2mm_P5.08mm_Vertical" V 4830 2900 50  0001 C CNN
+F 3 "https://eu.mouser.com/datasheet/2/219/MOS-16613.pdf" H 4900 2900 50  0001 C CNN
 	1    4900 2900
 	1    0    0    -1
@@
 F 0 "C33" H 5375 3200 50  0000 L CNN
 F 1 "4.7 nF" H 5375 3000 50  0000 L CNN
-F 2 "" H 5388 2950 50  0001 C CNN
-F 3 "" H 5350 3100 50  0001 C CNN
+F 2 "Capacitors_THT:C_Axial_L5.1mm_D3.1mm_P10.00mm_Horizontal" H 5388 2950 50  0001 C CNN
+F 3 "https://eu.mouser.com/datasheet/2/212/KEM_C1046_AXIAL_MOLDED_X7R-1145195.pdf" H 5350 3100 50  0001 C CNN
 	1    5350 3100
 	0    1    1    0
@@
 F 0 "C34" H 5375 3600 50  0000 L CNN
 F 1 "4.7 nF" H 5375 3400 50  0000 L CNN
-F 2 "" H 5388 3350 50  0001 C CNN
-F 3 "" H 5350 3500 50  0001 C CNN
+F 2 "Capacitors_THT:C_Axial_L5.1mm_D3.1mm_P10.00mm_Horizontal" H 5388 3350 50  0001 C CNN
+F 3 "https://eu.mouser.com/datasheet/2/212/KEM_C1046_AXIAL_MOLDED_X7R-1145195.pdf" H 5350 3500 50  0001 C CNN
 	1    5350 3500
 	0    1    1    0
@@
 F 0 "R36" V 5780 3300 50  0000 C CNN
 F 1 "62k" V 5700 3300 50  0000 C CNN
-F 2 "" V 5630 3300 50  0001 C CNN
-F 3 "" H 5700 3300 50  0001 C CNN
+F 2 "Resistors_THT:R_Axial_DIN0309_L9.0mm_D3.2mm_P5.08mm_Vertical" V 5630 3300 50  0001 C CNN
+F 3 "https://eu.mouser.com/datasheet/2/219/MOS-16613.pdf" H 5700 3300 50  0001 C CNN
 	1    5700 3300
 	1    0    0    -1
@@
 F 0 "U8" H 6150 3200 50  0000 L CNN
 F 1 "TL074" H 6150 2800 50  0000 L CNN
-F 2 "" H 6100 3100 50  0001 C CNN
+F 2 "TL074:DIL14" H 6100 3100 50  0001 C CNN
 F 3 "" H 6200 3200 50  0001 C CNN
 	4    6150 3000

Commit message: Shiii ir 5. iteraacija manai platei - layouts
Parts:
- C31, C32, C33, C34: footprint Capacitors_THT:C_Axial_L5.1mm_D3.1mm_P10.00mm_Horizontal -> Capacitors_SMD:C_0805_HandSoldering
- R31, R32, R33, R34, R35, R36: footprint Resistors_THT:R_Axial_DIN0309_L9.0mm_D3.2mm_P5.08mm_Vertical -> Resistors_SMD:R_0805_HandSoldering
- U8: footprint TL074:DIL14 -> TL074:SO14
Changed lines of the file:
@@
 EESchema Schematic File Version 2
+LIBS:Kursa_darbs_Klavs_Ozols-rescue
 LIBS:power
 LIBS:device
@@
 F 0 "U8" H 3850 3300 50  0000 L CNN
 F 1 "TL074" H 3850 2900 50  0000 L CNN
-F 2 "TL074:DIL14" H 3800 3200 50  0001 C CNN
+F 2 "TL074:SO14" H 3800 3200 50  0001 C CNN
 F 3 "" H 3900 3300 50  0001 C CNN
 	3    3850 3100
@@
 F 0 "R31" V 2430 3200 50  0000 C CNN
 F 1 "6.8k" V 2350 3200 50  0000 C CNN
-F 2 "Resistors_THT:R_Axial_DIN0309_L9.0mm_D3.2mm_P5.08mm_Vertical" V 2280 3200 50  0001 C CNN
-F 3 "https://eu.mouser.com/datasheet/2/219/MOS-16613.pdf" H 2350 3200 50  0001 C CNN
+F 2 "Resistors_SMD:R_0805_HandSoldering" V 2280 3200 50  0001 C CNN
+F 3 "https://eu.mouser.com/datasheet/2/219/RN73-11994.pdf" H 2350 3200 50  0001 C CNN
 	1    2350 3200
 	0    1    1    0
@@
 F 0 "R32" V 2680 3000 50  0000 C CNN
 F 1 "5.1k" V 2600 3000 50  0000 C CNN
-F 2 "Resistors_THT:R_Axial_DIN0309_L9.0mm_D3.2mm_P5.08mm_Vertical" V 2530 3000 50  0001 C CNN
-F 3 "https://eu.mouser.com/datasheet/2/219/MOS-16613.pdf" H 2600 3000 50  0001 C CNN
+F 2 "Resistors_SMD:R_0805_HandSoldering" V 2530 3000 50  0001 C CNN
+F 3 "https://eu.mouser.com/datasheet/2/219/RN73-11994.pdf" H 2600 3000 50  0001 C CNN
 	1    2600 3000
 	1    0    0    -1
@@
 F 0 "C31" H 3075 3300 50  0000 L CNN
 F 1 "4.7 nF" H 3075 3100 50  0000 L CNN
-F 2 "Capacitors_THT:C_Axial_L5.1mm_D3.1mm_P10.00mm_Horizontal" H 3088 3050 50  0001 C CNN
-F 3 "https://eu.mouser.com/datasheet/2/212/KEM_C1046_AXIAL_MOLDED_X7R-1145195.pdf" H 3050 3200 50  0001 C CNN
+F 2 "Capacitors_SMD:C_0805_HandSoldering" H 3088 3050 50  0001 C CNN
+F 3 "https://eu.mouser.com/datasheet/2/427/vjcommercialseries-222796.pdf" H 3050 3200 50  0001 C CNN
 	1    3050 3200
 	0    1    1    0
@@
 F 0 "C32" H 3075 3700 50  0000 L CNN
 F 1 "4.7 nF" H 3075 3500 50  0000 L CNN
-F 2 "Capacitors_THT:C_Axial_L5.1mm_D3.1mm_P10.00mm_Horizontal" H 3088 3450 50  0001 C CNN
-F 3 "https://eu.mouser.com/datasheet/2/212/KEM_C1046_AXIAL_MOLDED_X7R-1145195.pdf" H 3050 3600 50  0001 C CNN
+F 2 "Capacitors_SMD:C_0805_HandSoldering" H 3088 3450 50  0001 C CNN
+F 3 "https://eu.mouser.com/datasheet/2/427/vjcommercialseries-222796.pdf" H 3050 3600 50  0001 C CNN
 	1    3050 3600
 	0    1    1    0
@@
 F 0 "R33" V 3480 3400 50  0000 C CNN
 F 1 "62k" V 3400 3400 50  0000 C CNN
-F 2 "Resistors_THT:R_Axial_DIN0309_L9.0mm_D3.2mm_P5.08mm_Vertical" V 3330 3400 50  0001 C CNN
-F 3 "https://eu.mouser.com/datasheet/2/219/MOS-16613.pdf" H 3400 3400 50  0001 C CNN
+F 2 "Resistors_SMD:R_0805_HandSoldering" V 3330 3400 50  0001 C CNN
+F 3 "https://eu.mouser.com/datasheet/2/219/RN73-11994.pdf" H 3400 3400 50  0001 C CNN
 	1    3400 3400
 	1    0    0    -1
@@
 F 0 "R34" V 4730 3100 50  0000 C CNN
 F 1 "6.8k" V 4650 3100 50  0000 C CNN
-F 2 "Resistors_THT:R_Axial_DIN0309_L9.0mm_D3.2mm_P5.08mm_Vertical" V 4580 3100 50  0001 C CNN
-F 3 "https://eu.mouser.com/datasheet/2/219/MOS-16613.pdf" H 4650 3100 50  0001 C CNN
+F 2 "Resistors_SMD:R_0805_HandSoldering" V 4580 3100 50  0001 C CNN
+F 3 "https://eu.mouser.com/datasheet/2/219/RN73-11994.pdf" H 4650 3100 50  0001 C CNN
 	1    4650 3100
 	0    1    1    0
@@
 F 0 "R35" V 4980 2900 50  0000 C CNN
 F 1 "5.1k" V 4900 2900 50  0000 C CNN
-F 2 "Resistors_THT:R_Axial_DIN0309_L9.0mm_D3.2mm_P5.08mm_Vertical" V 4830 2900 50  0001 C CNN
-F 3 "https://eu.mouser.com/datasheet/2/219/MOS-16613.pdf" H 4900 2900 50  0001 C CNN
+F 2 "Resistors_SMD:R_0805_HandSoldering" V 4830 2900 50  0001 C CNN
+F 3 "https://eu.mouser.com/datasheet/2/219/RN73-11994.pdf" H 4900 2900 50  0001 C CNN
 	1    4900 2900
 	1    0    0    -1
@@
 F 0 "C33" H 5375 3200 50  0000 L CNN
 F 1 "4.7 nF" H 5375 3000 50  0000 L CNN
-F 2 "Capacitors_THT:C_Axial_L5.1mm_D3.1mm_P10.00mm_Horizontal" H 5388 2950 50  0001 C CNN
-F 3 "https://eu.mouser.com/datasheet/2/212/KEM_C1046_AXIAL_MOLDED_X7R-1145195.pdf" H 5350 3100 50  0001 C CNN
+F 2 "Capacitors_SMD:C_0805_HandSoldering" H 5388 2950 50  0001 C CNN
+F 3 "https://eu.mouser.com/datasheet/2/427/vjcommercialseries-222796.pdf" H 5350 3100 50  0001 C CNN
 	1    5350 3100
 	0    1    1    0
@@
 F 0 "C34" H 5375 3600 50  0000 L CNN
 F 1 "4.7 nF" H 5375 3400 50  0000 L CNN
-F 2 "Capacitors_THT:C_Axial_L5.1mm_D3.1mm_P10.00mm_Horizontal" H 5388 3350 50  0001 C CNN
-F 3 "https://eu.mouser.com/datasheet/2/212/KEM_C1046_AXIAL_MOLDED_X7R-1145195.pdf" H 5350 3500 50  0001 C CNN
+F 2 "Capacitors_SMD:C_0805_HandSoldering" H 5388 3350 50  0001 C CNN
+F 3 "https://eu.mouser.com/datasheet/2/427/vjcommercialseries-222796.pdf" H 5350 3500 50  0001 C CNN
 	1    5350 3500
 	0    1    1    0
@@
 F 0 "R36" V 5780 3300 50  0000 C CNN
 F 1 "62k" V 5700 3300 50  0000 C CNN
-F 2 "Resistors_THT:R_Axial_DIN0309_L9.0mm_D3.2mm_P5.08mm_Vertical" V 5630 3300 50  0001 C CNN
-F 3 "https://eu.mouser.com/datasheet/2/219/MOS-16613.pdf" H 5700 3300 50  0001 C CNN
+F 2 "Resistors_SMD:R_0805_HandSoldering" V 5630 3300 50  0001 C CNN
+F 3 "https://eu.mouser.com/datasheet/2/219/RN73-11994.pdf" H 5700 3300 50  0001 C CNN
 	1    5700 3300
 	1    0    0    -1
@@
 F 0 "U8" H 6150 3200 50  0000 L CNN
 F 1 "TL074" H 6150 2800 50  0000 L CNN
-F 2 "TL074:DIL14" H 6100 3100 50  0001 C CNN
+F 2 "TL074:SO14" H 6100 3100 50  0001 C CNN
 F 3 "" H 6200 3200 50  0001 C CNN
 	4    6150 3000
