File: Kursa_darbs_Klavs_Ozols/Filter8.sch (KiCad schematic (older format))
At the start: 11 parts, among them U9 TL074

Commit message: Shii ir kursa darba 3. iteraacija
Parts:
- C39, C40, C41, C42: footprint (none) -> Capacitors_THT:C_Axial_L5.1mm_D3.1mm_P10.00mm_Horizontal
- R43, R44, R45, R46, R47, R48: footprint (none) -> Resistors_THT:R_Axial_DIN0309_L9.0mm_D3.2mm_P5.08mm_Vertical
- U9: footprint (none) -> TL074:DIL14
Changed lines of the file:
@@
 F 0 "U9" H 4100 3800 50  0000 L CNN
 F 1 "TL074" H 4100 3400 50  0000 L CNN
-F 2 "" H 4050 3700 50  0001 C CNN
+F 2 "TL074:DIL14" H 4050 3700 50  0001 C CNN
 F 3 "" H 4150 3800 50  0001 C CNN
 	3    4100 3600
@@
 F 0 "R43" V 2930 3700 50  0000 C CNN
 F 1 "6.8k" V 2850 3700 50  0000 C CNN
-F 2 "" V 2780 3700 50  0001 C CNN
-F 3 "" H 2850 3700 50  0001 C CNN
+F 2 "Resistors_THT:R_Axial_DIN0309_L9.0mm_D3.2mm_P5.08mm_Vertical" V 2780 3700 50  0001 C CNN
+F 3 "https://eu.mouser.com/datasheet/2/219/MOS-16613.pdf" H 2850 3700 50  0001 C CNN
 	1    2850 3700
 	0    1    1    0
@@
 F 0 "R44" V 3180 3450 50  0000 C CNN
 F 1 "5.1k" V 3100 3450 50  0000 C CNN
-F 2 "" V 3030 3450 50  0001 C CNN
-F 3 "" H 3100 3450 50  0001 C CNN
+F 2 "Resistors_THT:R_Axial_DIN0309_L9.0mm_D3.2mm_P5.08mm_Vertical" V 3030 3450 50  0001 C CNN
+F 3 "https://eu.mouser.com/datasheet/2/219/MOS-16613.pdf" H 3100 3450 50  0001 C CNN
 	1    3100 3450
 	1    0    0    -1
@@
 F 0 "C39" H 3375 3800 50  0000 L CNN
 F 1 "1nF" H 3375 3600 50  0000 L CNN
-F 2 "" H 3388 3550 50  0001 C CNN
-F 3 "" H 3350 3700 50  0001 C CNN
+F 2 "Capacitors_THT:C_Axial_L5.1mm_D3.1mm_P10.00mm_Horizontal" H 3388 3550 50  0001 C CNN
+F 3 "https://eu.mouser.com/datasheet/2/212/KEM_C1046_AXIAL_MOLDED_X7R-1145195.pdf" H 3350 3700 50  0001 C CNN
 	1    3350 3700
 	0    1    1    0
@@
 F 0 "C40" H 3375 4200 50  0000 L CNN
 F 1 "1nF" H 3375 4000 50  0000 L CNN
-F 2 "" H 3388 3950 50  0001 C CNN
-F 3 "" H 3350 4100 50  0001 C CNN
+F 2 "Capacitors_THT:C_Axial_L5.1mm_D3.1mm_P10.00mm_Horizontal" H 3388 3950 50  0001 C CNN
+F 3 "https://eu.mouser.com/datasheet/2/212/KEM_C1046_AXIAL_MOLDED_X7R-1145195.pdf" H 3350 4100 50  0001 C CNN
 	1    3350 4100
 	0    1    1    0
@@
 F 0 "R45" V 3730 3900 50  0000 C CNN
 F 1 "62k" V 3650 3900 50  0000 C CNN
-F 2 "" V 3580 3900 50  0001 C CNN
-F 3 "" H 3650 3900 50  0001 C CNN
+F 2 "Resistors_THT:R_Axial_DIN0309_L9.0mm_D3.2mm_P5.08mm_Vertical" V 3580 3900 50  0001 C CNN
+F 3 "https://eu.mouser.com/datasheet/2/219/MOS-16613.pdf" H 3650 3900 50  0001 C CNN
 	1    3650 3900
 	1    0    0    -1
@@
 F 0 "R46" V 5180 3600 50  0000 C CNN
 F 1 "6.8k" V 5100 3600 50  0000 C CNN
-F 2 "" V 5030 3600 50  0001 C CNN
-F 3 "" H 5100 3600 50  0001 C CNN
+F 2 "Resistors_THT:R_Axial_DIN0309_L9.0mm_D3.2mm_P5.08mm_Vertical" V 5030 3600 50  0001 C CNN
+F 3 "https://eu.mouser.com/datasheet/2/219/MOS-16613.pdf" H 5100 3600 50  0001 C CNN
 	1    5100 3600
 	0    1    1    0
@@
 F 0 "R47" V 5430 3350 50  0000 C CNN
 F 1 "5.1k" V 5350 3350 50  0000 C CNN
-F 2 "" V 5280 3350 50  0001 C CNN
-F 3 "" H 5350 3350 50  0001 C CNN
+F 2 "Resistors_THT:R_Axial_DIN0309_L9.0mm_D3.2mm_P5.08mm_Vertical" V 5280 3350 50  0001 C CNN
+F 3 "https://eu.mouser.com/datasheet/2/219/MOS-16613.pdf" H 5350 3350 50  0001 C CNN
 	1    5350 3350
 	1    0    0    -1
@@
 F 0 "C41" H 5625 3700 50  0000 L CNN
 F 1 "1nF" H 5625 3500 50  0000 L CNN
-F 2 "" H 5638 3450 50  0001 C CNN
-F 3 "" H 5600 3600 50  0001 C CNN
+F 2 "Capacitors_THT:C_Axial_L5.1mm_D3.1mm_P10.00mm_Horizontal" H 5638 3450 50  0001 C CNN
+F 3 "https://eu.mouser.com/datasheet/2/212/KEM_C1046_AXIAL_MOLDED_X7R-1145195.pdf" H 5600 3600 50  0001 C CNN
 	1    5600 3600
 	0    1    1    0
@@
 F 0 "C42" H 5625 4100 50  0000 L CNN
 F 1 "1nF" H 5625 3900 50  0000 L CNN
-F 2 "" H 5638 3850 50  0001 C CNN
-F 3 "" H 5600 4000 50  0001 C CNN
+F 2 "Capacitors_THT:C_Axial_L5.1mm_D3.1mm_P10.00mm_Horizontal" H 5638 3850 50  0001 C CNN
+F 3 "https://eu.mouser.com/datasheet/2/212/KEM_C1046_AXIAL_MOLDED_X7R-1145195.pdf" H 5600 4000 50  0001 C CNN
 	1    5600 4000
 	0    1    1    0
@@
 F 0 "R48" V 5980 3800 50  0000 C CNN
 F 1 "62k" V 5900 3800 50  0000 C CNN
-F 2 "" V 5830 3800 50  0001 C CNN
-F 3 "" H 5900 3800 50  0001 C CNN
+F 2 "Resistors_THT:R_Axial_DIN0309_L9.0mm_D3.2mm_P5.08mm_Vertical" V 5830 3800 50  0001 C CNN
+F 3 "https://eu.mouser.com/datasheet/2/219/MOS-16613.pdf" H 5900 3800 50  0001 C CNN
 	1    5900 3800
 	1    0    0    -1
@@
 F 0 "U9" H 6350 3700 50  0000 L CNN
 F 1 "TL074" H 6350 3300 50  0000 L CNN
-F 2 "" H 6300 3600 50  0001 C CNN
+F 2 "TL074:DIL14" H 6300 3600 50  0001 C CNN
 F 3 "" H 6400 3700 50  0001 C CNN
 	4    6350 3500

Commit message: Shiii ir 5. iteraacija manai platei - layouts
Parts:
- C39, C40, C41, C42: footprint Capacitors_THT:C_Axial_L5.1mm_D3.1mm_P10.00mm_Horizontal -> Capacitors_SMD:C_0805_HandSoldering
- R43, R44, R45, R46, R47, R48: footprint Resistors_THT:R_Axial_DIN0309_L9.0mm_D3.2mm_P5.08mm_Vertical -> Resistors_SMD:R_0805_HandSoldering
- U9: footprint TL074:DIL14 -> TL074:SO14
Changed lines of the file:
@@
 EESchema Schematic File Version 2
+LIBS:Kursa_darbs_Klavs_Ozols-rescue
 LIBS:power
 LIBS:device
@@
 F 0 "U9" H 4100 3800 50  0000 L CNN
 F 1 "TL074" H 4100 3400 50  0000 L CNN
-F 2 "TL074:DIL14" H 4050 3700 50  0001 C CNN
+F 2 "TL074:SO14" H 4050 3700 50  0001 C CNN
 F 3 "" H 4150 3800 50  0001 C CNN
 	3    4100 3600
@@
 F 0 "R43" V 2930 3700 50  0000 C CNN
 F 1 "6.8k" V 2850 3700 50  0000 C CNN
-F 2 "Resistors_THT:R_Axial_DIN0309_L9.0mm_D3.2mm_P5.08mm_Vertical" V 2780 3700 50  0001 C CNN
-F 3 "https://eu.mouser.com/datasheet/2/219/MOS-16613.pdf" H 2850 3700 50  0001 C CNN
+F 2 "Resistors_SMD:R_0805_HandSoldering" V 2780 3700 50  0001 C CNN
+F 3 "https://eu.mouser.com/datasheet/2/219/RN73-11994.pdf" H 2850 3700 50  0001 C CNN
 	1    2850 3700
 	0    1    1    0
@@
 F 0 "R44" V 3180 3450 50  0000 C CNN
 F 1 "5.1k" V 3100 3450 50  0000 C CNN
-F 2 "Resistors_THT:R_Axial_DIN0309_L9.0mm_D3.2mm_P5.08mm_Vertical" V 3030 3450 50  0001 C CNN
-F 3 "https://eu.mouser.com/datasheet/2/219/MOS-16613.pdf" H 3100 3450 50  0001 C CNN
+F 2 "Resistors_SMD:R_0805_HandSoldering" V 3030 3450 50  0001 C CNN
+F 3 "https://eu.mouser.com/datasheet/2/219/RN73-11994.pdf" H 3100 3450 50  0001 C CNN
 	1    3100 3450
 	1    0    0    -1
@@
 F 0 "C39" H 3375 3800 50  0000 L CNN
 F 1 "1nF" H 3375 3600 50  0000 L CNN
-F 2 "Capacitors_THT:C_Axial_L5.1mm_D3.1mm_P10.00mm_Horizontal" H 3388 3550 50  0001 C CNN
-F 3 "https://eu.mouser.com/datasheet/2/212/KEM_C1046_AXIAL_MOLDED_X7R-1145195.pdf" H 3350 3700 50  0001 C CNN
+F 2 "Capacitors_SMD:C_0805_HandSoldering" H 3388 3550 50  0001 C CNN
+F 3 "https://eu.mouser.com/datasheet/2/427/vjcommercialseries-222796.pdf" H 3350 3700 50  0001 C CNN
 	1    3350 3700
 	0    1    1    0
@@
 F 0 "C40" H 3375 4200 50  0000 L CNN
 F 1 "1nF" H 3375 4000 50  0000 L CNN
-F 2 "Capacitors_THT:C_Axial_L5.1mm_D3.1mm_P10.00mm_Horizontal" H 3388 3950 50  0001 C CNN
-F 3 "https://eu.mouser.com/datasheet/2/212/KEM_C1046_AXIAL_MOLDED_X7R-1145195.pdf" H 3350 4100 50  0001 C CNN
+F 2 "Capacitors_SMD:C_0805_HandSoldering" H 3388 3950 50  0001 C CNN
+F 3 "https://eu.mouser.com/datasheet/2/427/vjcommercialseries-222796.pdf" H 3350 4100 50  0001 C CNN
 	1    3350 4100
 	0    1    1    0
@@
 F 0 "R45" V 3730 3900 50  0000 C CNN
 F 1 "62k" V 3650 3900 50  0000 C CNN
-F 2 "Resistors_THT:R_Axial_DIN0309_L9.0mm_D3.2mm_P5.08mm_Vertical" V 3580 3900 50  0001 C CNN
-F 3 "https://eu.mouser.com/datasheet/2/219/MOS-16613.pdf" H 3650 3900 50  0001 C CNN
+F 2 "Resistors_SMD:R_0805_HandSoldering" V 3580 3900 50  0001 C CNN
+F 3 "https://eu.mouser.com/datasheet/2/219/RN73-11994.pdf" H 3650 3900 50  0001 C CNN
 	1    3650 3900
 	1    0    0    -1
@@
 F 0 "R46" V 5180 3600 50  0000 C CNN
 F 1 "6.8k" V 5100 3600 50  0000 C CNN
-F 2 "Resistors_THT:R_Axial_DIN0309_L9.0mm_D3.2mm_P5.08mm_Vertical" V 5030 3600 50  0001 C CNN
-F 3 "https://eu.mouser.com/datasheet/2/219/MOS-16613.pdf" H 5100 3600 50  0001 C CNN
+F 2 "Resistors_SMD:R_0805_HandSoldering" V 5030 3600 50  0001 C CNN
+F 3 "https://eu.mouser.com/datasheet/2/219/RN73-11994.pdf" H 5100 3600 50  0001 C CNN
 	1    5100 3600
 	0    1    1    0
@@
 F 0 "R47" V 5430 3350 50  0000 C CNN
 F 1 "5.1k" V 5350 3350 50  0000 C CNN
-F 2 "Resistors_THT:R_Axial_DIN0309_L9.0mm_D3.2mm_P5.08mm_Vertical" V 5280 3350 50  0001 C CNN
-F 3 "https://eu.mouser.com/datasheet/2/219/MOS-16613.pdf" H 5350 3350 50  0001 C CNN
+F 2 "Resistors_SMD:R_0805_HandSoldering" V 5280 3350 50  0001 C CNN
+F 3 "https://eu.mouser.com/datasheet/2/219/RN73-11994.pdf" H 5350 3350 50  0001 C CNN
 	1    5350 3350
 	1    0    0    -1
@@
 F 0 "C41" H 5625 3700 50  0000 L CNN
 F 1 "1nF" H 5625 3500 50  0000 L CNN
-F 2 "Capacitors_THT:C_Axial_L5.1mm_D3.1mm_P10.00mm_Horizontal" H 5638 3450 50  0001 C CNN
-F 3 "https://eu.mouser.com/datasheet/2/212/KEM_C1046_AXIAL_MOLDED_X7R-1145195.pdf" H 5600 3600 50  0001 C CNN
+F 2 "Capacitors_SMD:C_0805_HandSoldering" H 5638 3450 50  0001 C CNN
+F 3 "https://eu.mouser.com/datasheet/2/427/vjcommercialseries-222796.pdf" H 5600 3600 50  0001 C CNN
 	1    5600 3600
 	0    1    1    0
@@
 F 0 "C42" H 5625 4100 50  0000 L CNN
 F 1 "1nF" H 5625 3900 50  0000 L CNN
-F 2 "Capacitors_THT:C_Axial_L5.1mm_D3.1mm_P10.00mm_Horizontal" H 5638 3850 50  0001 C CNN
-F 3 "https://eu.mouser.com/datasheet/2/212/KEM_C1046_AXIAL_MOLDED_X7R-1145195.pdf" H 5600 4000 50  0001 C CNN
+F 2 "Capacitors_SMD:C_0805_HandSoldering" H 5638 3850 50  0001 C CNN
+F 3 "https://eu.mouser.com/datasheet/2/427/vjcommercialseries-222796.pdf" H 5600 4000 50  0001 C CNN
 	1    5600 4000
 	0    1    1    0
@@
 F 0 "R48" V 5980 3800 50  0000 C CNN
 F 1 "62k" V 5900 3800 50  0000 C CNN
-F 2 "Resistors_THT:R_Axial_DIN0309_L9.0mm_D3.2mm_P5.08mm_Vertical" V 5830 3800 50  0001 C CNN
-F 3 "https://eu.mouser.com/datasheet/2/219/MOS-16613.pdf" H 5900 3800 50  0001 C CNN
+F 2 "Resistors_SMD:R_0805_HandSoldering" V 5830 3800 50  0001 C CNN
+F 3 "https://eu.mouser.com/datasheet/2/219/RN73-11994.pdf" H 5900 3800 50  0001 C CNN
 	1    5900 3800
 	1    0    0    -1
@@
 F 0 "U9" H 6350 3700 50  0000 L CNN
 F 1 "TL074" H 6350 3300 50  0000 L CNN
-F 2 "TL074:DIL14" H 6300 3600 50  0001 C CNN
+F 2 "TL074:SO14" H 6300 3600 50  0001 C CNN
 F 3 "" H 6400 3700 50  0001 C CNN
 	4    6350 3500
