File: Kursa_darbs_Klavs_Ozols/Filter4.sch (KiCad schematic (older format))
At the start: 11 parts, among them U7 TL074

Commit message: Shii ir 2. iteraacija kursa darbam!
Connections:
- net Audio500Hz: now also R24.1; no longer R24.2
- net at C24.1, R22.2, U7.8: now also R21.1; no longer R21.2
- net at C23.1, U7.9 (-): now also R21.2; no longer R21.1
- net at C25.1, U7.13 (-): now also R24.2; no longer R24.1
Changed lines of the file:
@@
 F 3 "" H 3050 2650 50  0001 C CNN
 	1    3050 2650
-	1    0    0    -1
+	0    1    1    0
 $EndComp
 $Comp
@@
 	4050 2800 2900 2800
 Wire Wire Line
-	4050 2400 4050 2800
+	4050 2300 4050 2800
 Wire Wire Line
 	4050 2400 3850 2400
@@
 F 3 "" H 4200 2450 50  0001 C CNN
 	1    4200 2450
-	0    1    1    0
+	-1   0    0    1
 $EndComp
 $Comp
@@
 F 3 "" H 4400 2200 50  0001 C CNN
 	1    4400 2200
-	1    0    0    -1
+	0    1    1    0
 $EndComp
 $Comp
@@
 F 3 "" H 4850 2600 50  0001 C CNN
 	1    4850 2600
-	1    0    0    -1
+	0    1    1    0
 $EndComp
 Wire Wire Line
@@
 	5150 3200 5150 2650
 Connection ~ 3400 3200
-Connection ~ 4050 2450
 Wire Wire Line
 	2050 2500 1750 2500
@@
 Wire Wire Line
 	3400 2700 3450 2700
+Wire Wire Line
+	2900 2650 2900 2550
+Wire Wire Line
+	2900 2550 3050 2550
+Wire Wire Line
+	3050 2550 3050 2500
+Wire Wire Line
+	3200 2650 3200 2750
+Wire Wire Line
+	3200 2750 3050 2750
+Wire Wire Line
+	3050 2750 3050 2800
+Wire Wire Line
+	4200 2300 4050 2300
+Connection ~ 4050 2400
+Wire Wire Line
+	4200 2600 4350 2600
+Wire Wire Line
+	4350 2600 4350 2450
+Wire Wire Line
+	4400 2050 4400 2100
+Wire Wire Line
+	4400 2100 4550 2100
+Wire Wire Line
+	4550 2100 4550 2200
+Wire Wire Line
+	4250 2200 4250 2300
+Wire Wire Line
+	4250 2300 4300 2300
+Wire Wire Line
+	4300 2300 4300 2350
+Wire Wire Line
+	4300 2350 4400 2350
+Wire Wire Line
+	4700 2600 4700 2550
+Wire Wire Line
+	4700 2550 4850 2550
+Wire Wire Line
+	4850 2550 4850 2450
+Wire Wire Line
+	5000 2600 5000 2750
+Wire Wire Line
+	5000 2750 4850 2750
 $EndSCHEMATC

Commit message: Shii ir kursa darba 3. iteraacija
Parts:
- C23, C24, C25, C26: footprint (none) -> Capacitors_THT:C_Axial_L5.1mm_D3.1mm_P10.00mm_Horizontal
- R19, R20, R21, R22, R23, R24: footprint (none) -> Resistors_THT:R_Axial_DIN0309_L9.0mm_D3.2mm_P5.08mm_Vertical
- U7: footprint (none) -> TL074:DIL14
Changed lines of the file:
@@
 F 0 "U7" H 3550 2600 50  0000 L CNN
 F 1 "TL074" H 3550 2200 50  0000 L CNN
-F 2 "" H 3500 2500 50  0001 C CNN
+F 2 "TL074:DIL14" H 3500 2500 50  0001 C CNN
 F 3 "" H 3600 2600 50  0001 C CNN
 	3    3550 2400
@@
 F 0 "U7" H 5250 2550 50  0000 L CNN
 F 1 "TL074" H 5250 2150 50  0000 L CNN
-F 2 "" H 5200 2450 50  0001 C CNN
+F 2 "TL074:DIL14" H 5200 2450 50  0001 C CNN
 F 3 "" H 5300 2550 50  0001 C CNN
 	4    5250 2350
@@
 F 0 "R19" V 2280 2500 50  0000 C CNN
 F 1 "6.8k" V 2200 2500 50  0000 C CNN
-F 2 "" V 2130 2500 50  0001 C CNN
-F 3 "" H 2200 2500 50  0001 C CNN
+F 2 "Resistors_THT:R_Axial_DIN0309_L9.0mm_D3.2mm_P5.08mm_Vertical" V 2130 2500 50  0001 C CNN
+F 3 "https://eu.mouser.com/datasheet/2/219/MOS-16613.pdf" H 2200 2500 50  0001 C CNN
 	1    2200 2500
 	0    1    1    0
@@
 F 0 "R21" V 3130 2650 50  0000 C CNN
 F 1 "62k" V 3050 2650 50  0000 C CNN
-F 2 "" V 2980 2650 50  0001 C CNN
-F 3 "" H 3050 2650 50  0001 C CNN
+F 2 "Resistors_THT:R_Axial_DIN0309_L9.0mm_D3.2mm_P5.08mm_Vertical" V 2980 2650 50  0001 C CNN
+F 3 "https://eu.mouser.com/datasheet/2/219/MOS-16613.pdf" H 3050 2650 50  0001 C CNN
 	1    3050 2650
 	0    1    1    0
@@
 F 0 "C23" H 2775 2600 50  0000 L CNN
 F 1 "22nF" H 2775 2400 50  0000 L CNN
-F 2 "" H 2788 2350 50  0001 C CNN
-F 3 "" H 2750 2500 50  0001 C CNN
+F 2 "Capacitors_THT:C_Axial_L5.1mm_D3.1mm_P10.00mm_Horizontal" H 2788 2350 50  0001 C CNN
+F 3 "https://eu.mouser.com/datasheet/2/212/KEM_C1046_AXIAL_MOLDED_X7R-1145195.pdf" H 2750 2500 50  0001 C CNN
 	1    2750 2500
 	0    1    1    0
@@
 F 0 "C24" H 2775 2900 50  0000 L CNN
 F 1 "22nF" H 2775 2700 50  0000 L CNN
-F 2 "" H 2788 2650 50  0001 C CNN
-F 3 "" H 2750 2800 50  0001 C CNN
+F 2 "Capacitors_THT:C_Axial_L5.1mm_D3.1mm_P10.00mm_Horizontal" H 2788 2650 50  0001 C CNN
+F 3 "https://eu.mouser.com/datasheet/2/212/KEM_C1046_AXIAL_MOLDED_X7R-1145195.pdf" H 2750 2800 50  0001 C CNN
 	1    2750 2800
 	0    1    1    0
@@
 F 0 "R20" V 2530 2250 50  0000 C CNN
 F 1 "5.1k" V 2450 2250 50  0000 C CNN
-F 2 "" V 2380 2250 50  0001 C CNN
-F 3 "" H 2450 2250 50  0001 C CNN
+F 2 "Resistors_THT:R_Axial_DIN0309_L9.0mm_D3.2mm_P5.08mm_Vertical" V 2380 2250 50  0001 C CNN
+F 3 "https://eu.mouser.com/datasheet/2/219/MOS-16613.pdf" H 2450 2250 50  0001 C CNN
 	1    2450 2250
 	1    0    0    -1
@@
 F 0 "R22" V 4280 2450 50  0000 C CNN
 F 1 "6.8k" V 4200 2450 50  0000 C CNN
-F 2 "" V 4130 2450 50  0001 C CNN
-F 3 "" H 4200 2450 50  0001 C CNN
+F 2 "Resistors_THT:R_Axial_DIN0309_L9.0mm_D3.2mm_P5.08mm_Vertical" V 4130 2450 50  0001 C CNN
+F 3 "https://eu.mouser.com/datasheet/2/219/MOS-16613.pdf" H 4200 2450 50  0001 C CNN
 	1    4200 2450
 	-1   0    0    1
@@
 F 0 "C26" H 4625 2900 50  0000 L CNN
 F 1 "22nF" H 4625 2700 50  0000 L CNN
-F 2 "" H 4638 2650 50  0001 C CNN
-F 3 "" H 4600 2800 50  0001 C CNN
+F 2 "Capacitors_THT:C_Axial_L5.1mm_D3.1mm_P10.00mm_Horizontal" H 4638 2650 50  0001 C CNN
+F 3 "https://eu.mouser.com/datasheet/2/212/KEM_C1046_AXIAL_MOLDED_X7R-1145195.pdf" H 4600 2800 50  0001 C CNN
 	1    4600 2800
 	0    1    1    0
@@
 F 0 "C25" H 4625 2550 50  0000 L CNN
 F 1 "22nF" H 4625 2350 50  0000 L CNN
-F 2 "" H 4638 2300 50  0001 C CNN
-F 3 "" H 4600 2450 50  0001 C CNN
+F 2 "Capacitors_THT:C_Axial_L5.1mm_D3.1mm_P10.00mm_Horizontal" H 4638 2300 50  0001 C CNN
+F 3 "https://eu.mouser.com/datasheet/2/212/KEM_C1046_AXIAL_MOLDED_X7R-1145195.pdf" H 4600 2450 50  0001 C CNN
 	1    4600 2450
 	0    1    1    0
@@
 F 0 "R23" V 4480 2200 50  0000 C CNN
 F 1 "5.1k" V 4400 2200 50  0000 C CNN
-F 2 "" V 4330 2200 50  0001 C CNN
-F 3 "" H 4400 2200 50  0001 C CNN
+F 2 "Resistors_THT:R_Axial_DIN0309_L9.0mm_D3.2mm_P5.08mm_Vertical" V 4330 2200 50  0001 C CNN
+F 3 "https://eu.mouser.com/datasheet/2/219/MOS-16613.pdf" H 4400 2200 50  0001 C CNN
 	1    4400 2200
 	0    1    1    0
@@
 F 0 "R24" V 4930 2600 50  0000 C CNN
 F 1 "62k" V 4850 2600 50  0000 C CNN
-F 2 "" V 4780 2600 50  0001 C CNN
-F 3 "" H 4850 2600 50  0001 C CNN
+F 2 "Resistors_THT:R_Axial_DIN0309_L9.0mm_D3.2mm_P5.08mm_Vertical" V 4780 2600 50  0001 C CNN
+F 3 "https://eu.mouser.com/datasheet/2/219/MOS-16613.pdf" H 4850 2600 50  0001 C CNN
 	1    4850 2600
 	0    1    1    0

Commit message: Shiii ir 5. iteraacija manai platei - layouts
Parts:
- C23, C24, C25, C26: footprint Capacitors_THT:C_Axial_L5.1mm_D3.1mm_P10.00mm_Horizontal -> Capacitors_SMD:C_0805_HandSoldering
- R19, R20, R21, R22, R23, R24: footprint Resistors_THT:R_Axial_DIN0309_L9.0mm_D3.2mm_P5.08mm_Vertical -> Resistors_SMD:R_0805_HandSoldering
- U7: footprint TL074:DIL14 -> TL074:SO14
Connections:
- wire segments 48 -> 32
Other:
- moved on the sheet: C24, C25, C26, R21, R22, R23, R24, U7D

Commit message: Shis ir mans meeginaajums iztraseet plati ( nepabeigts- vajag paliidziibu)
Changed lines of the file:
@@
 	5050 1900 5050 2250
 Wire Wire Line
-	5050 1900 2050 1900
+	1950 1900 5050 1900
 Wire Wire Line
 	2450 2100 2450 1900
