File: Kursa_darbs_Klavs_Ozols/Kursa_darbs_Klavs_Ozols_2_ver.kicad_pcb (KiCad board)
At the start: 4 copper layers, 215 x 140 mm, 367 parts, among them J1 Barosana, J10 Conn_01x01, J11 Conn_01x01, J12 Conn_01x01, J13 Conn_01x01, J14 Conn_01x01, J15 Conn_01x01, J16 Conn_01x01, J17 Conn_01x01, J18 Conn_01x01, J19 Conn_01x01, J2 Audio-Jack-3, J20 Conn_01x01, J21 Conn_01x01, J22 Conn_01x01, J23 Conn_01x01, J24 Conn_01x01, J25 Conn_01x01, J26 Conn_01x01, J27 Conn_01x01, J28 Conn_01x01, J29 Conn_01x01, J3 Conn_01x01, J30 Conn_01x01, J31 Conn_01x01, J32 Conn_01x01, J33 Conn_01x01, J34 Conn_01x01, J35 Conn_01x01, J36 Conn_01x01, J37 Conn_01x01, J38 Conn_01x01, J39 Conn_01x01, J4 Conn_01x01, J40 Conn_01x01, J41 Conn_01x01, J42 Conn_01x01, J43 Conn_01x01, J44 Conn_01x01, J45 Conn_01x01, J46 Conn_01x01, J47 Conn_01x01, J48 Conn_01x01, J49 Conn_01x01, J5 Conn_01x01, J50 Conn_01x01, J51 Conn_01x01, J52 Conn_01x01, J6 Conn_01x01, J7 Conn_01x01, J8 Conn_01x01, J9 Conn_01x01, U1 TL074, U10 TL074, U11 TL074, U12 TL074, U13 LM3915, U14 LM3915, U15 LM3915, U16 LM3915, U17 LM3915, U18 LM3915, U19 LM317_TO3, U2 L7808, U20 LM3915, U21 LM3915, U22 LM3915, U3 ICL7660SIPAZ, U4 ICL7660SIPAZ, U5 ICL7660SIPAZ, U6 ICL7660SIPAZ, U7 TL074, U8 TL074, U9 TL074

Commit message: Kursa/Prakses darba pabeigtaa plates versija
Parts:
- removed J38, J39, J40, J41, J42, J43, J44, J45, J46, J47, J48, J49, J50, J51, J52: Conn_01x01, Measurement_Points:Measurement_Point_Round-TH_Small
- moved J26 172.3 mm to (289.1, 215.3)
- moved J14 157.0 mm to (250.2, 215.4)
- moved J20 154.9 mm to (279.5, 215.4)
- moved J27 154.2 mm to (298.9, 208.9)
- moved J24 152.8 mm to (221.7, 215.5)
- moved J23 149.0 mm to (221.8, 209.0)
- moved J31 143.3 mm to (185.2, 210.3)
- moved J13 143.2 mm to (240.6, 215.4)
- moved J11 142.5 mm to (249.8, 209.2)
- moved J33 142.3 mm to (176.1, 210.2)
- moved J30 132.5 mm to (194.3, 216.1)
- moved J21 130.3 mm to (230.9, 209.1)
- moved J19 129.0 mm to (279.6, 208.8)
- moved J18 127.8 mm to (269.8, 215.3)
- moved J22 125.3 mm to (231.0, 215.5)
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Connections:
- J11 pad 1: /10Hz-100nF/Audio10Hz -> /50
- J12 pad 1: /10Hz-100nF/Audio10Hz -> /200
- J13 pad 1: /50Hz - 220 nF/Audio50Hz -> /1k
- J14 pad 1: /50Hz - 220 nF/Audio50Hz -> /10k
- J18 pad 1: /200Hz - 47nF/Audio200Hz -> GND
- J19 pad 1: /200Hz - 47nF/Audio200Hz -> GND
- J20 pad 1: /500Hz - 22 nF/Audio500Hz -> GND
- J34 pad 1: /500Hz - 22 nF/Audio500Hz -> GND
Routing:
- net /All_Indicators/Turpinajums/LED_Supply: track 921.0 -> 0.00 mm
- net /+8V: track 582.7 -> 44.2 mm
- net /-8V: track 213.7 -> 7.68 mm
- net /-8V_2: track 215.6 -> 22.0 mm
- net /-8V_3: track 182.4 -> 28.1 mm
- net /-8V_1: track 324.0 -> 250.2 mm
- net GND: track 76.7 -> 7.36 mm
- net /10: track 71.0 -> 7.88 mm
- net /500Hz - 22 nF/Audio500Hz: track 67.9 -> 6.67 mm
- net /10Hz-100nF/Audio10Hz: track 62.0 -> 7.57 mm
- net /50Hz - 220 nF/Audio50Hz: track 63.3 -> 9.61 mm
- net /500: track 61.2 -> 14.0 mm
- net /2.5 kHz- 4.7 nF/Audio2.5kHz: track 53.0 -> 6.28 mm
- net /10 kHz - 1 nF/Audio10kHz: track 46.4 -> 7.28 mm
- net /4.5kHz - 2.2 nF/Audio4.5kHz: track 42.8 -> 6.78 mm
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