File: Kursa_darbs_Klavs_Ozols/Barosana.sch (KiCad schematic (older format))
At the start: 15 parts, among them U2 L7808, U3 ICL7660SIPAZ, U4 ICL7660SIPAZ, U5 ICL7660SIPAZ, U6 ICL7660SIPAZ

Commit message: Shiii ir 5. iteraacija manai platei - layouts
Parts:
- C10, C7, C8, C9: footprint Capacitors_THT:CP_Radial_D10.0mm_P5.00mm -> Capacitors_SMD:CP_Elec_4x5.8
- C11, C12, C13, C14: footprint Capacitors_THT:CP_Radial_D10.0mm_P5.00mm -> Capacitors_SMD:CP_Elec_10x10.5
- C5, C6: footprint Capacitors_THT:C_Axial_L3.8mm_D2.6mm_P7.50mm_Horizontal -> Capacitors_SMD:C_1210_HandSoldering
- U3, U4, U5, U6: footprint ICL7660SIPAZ:DIP254P762X533-8 -> Housings_SOIC:SOIC-8_3.9x4.9mm_Pitch1.27mm
Connections:
- net +8V_3 renamed GND
Changed lines of the file:
@@
 EESchema Schematic File Version 2
+LIBS:Kursa_darbs_Klavs_Ozols-rescue
 LIBS:power
 LIBS:device
@@
 F 0 "C5" H 1925 1500 50  0000 L CNN
 F 1 "100 nF" H 1925 1300 50  0000 L CNN
-F 2 "Capacitors_THT:C_Axial_L3.8mm_D2.6mm_P7.50mm_Horizontal" H 1938 1250 50  0001 C CNN
-F 3 "https://eu.mouser.com/datasheet/2/427/maseries-1211360.pdf" H 1900 1400 50  0001 C CNN
+F 2 "Capacitors_SMD:C_1210_HandSoldering" H 1938 1250 50  0001 C CNN
+F 3 "https://eu.mouser.com/datasheet/2/427/vjw1bcbascomseries-223529.pdf" H 1900 1400 50  0001 C CNN
 	1    1900 1400
 	1    0    0    -1
@@
 F 0 "C6" H 2875 1500 50  0000 L CNN
 F 1 "100 nF" H 2875 1300 50  0000 L CNN
-F 2 "Capacitors_THT:C_Axial_L3.8mm_D2.6mm_P7.50mm_Horizontal" H 2888 1250 50  0001 C CNN
-F 3 "https://eu.mouser.com/datasheet/2/427/maseries-1211360.pdf" H 2850 1400 50  0001 C CNN
+F 2 "Capacitors_SMD:C_1210_HandSoldering" H 2888 1250 50  0001 C CNN
+F 3 "https://eu.mouser.com/datasheet/2/427/vjw1bcbascomseries-223529.pdf" H 2850 1400 50  0001 C CNN
 	1    2850 1400
 	1    0    0    -1
@@
 F 0 "U3" H 4550 1950 50  0000 L BNN
 F 1 "ICL7660SIPAZ" H 4350 700 50  0000 L BNN
-F 2 "ICL7660SIPAZ:DIP254P762X533-8" H 4550 1450 50  0001 L BNN
-F 3 "Good" H 4550 1450 50  0001 L BNN
+F 2 "Housings_SOIC:SOIC-8_3.9x4.9mm_Pitch1.27mm" H 4550 1450 50  0001 L BNN
+F 3 "https://eu.mouser.com/datasheet/2/698/icl7660-1302119.pdf" H 4550 1450 50  0001 L BNN
 F 4 "ICL7660SIPAZ" H 4550 1450 50  0001 L BNN "Field4"
 F 5 "Intersil" H 4550 1450 50  0001 L BNN "Field5"
@@
 F 0 "C7" H 3575 1600 50  0000 L CNN
 F 1 "10 uF" H 3300 1400 50  0000 L CNN
-F 2 "Capacitors_THT:CP_Radial_D10.0mm_P5.00mm" H 3550 1500 50  0001 C CNN
-F 3 "https://eu.mouser.com/datasheet/2/293/e-upx-876312.pdf" H 3550 1500 50  0001 C CNN
+F 2 "Capacitors_SMD:CP_Elec_4x5.8" H 3550 1500 50  0001 C CNN
+F 3 "https://eu.mouser.com/datasheet/2/315/ABA0000C1251-1138508.pdf" H 3550 1500 50  0001 C CNN
 	1    3550 1500
 	1    0    0    -1
@@
 Connection ~ 2350 1800
 Wire Wire Line
-	3850 2050 3850 2300
-Wire Wire Line
-	3850 2300 5550 2300
+	3700 2300 5550 2300
 $Comp
 L CP1 C14
@@
 F 0 "C14" H 5875 1400 50  0000 L CNN
 F 1 "470 uF" H 5875 1200 50  0000 L CNN
-F 2 "Capacitors_THT:CP_Radial_D10.0mm_P5.00mm" H 5850 1300 50  0001 C CNN
+F 2 "Capacitors_SMD:CP_Elec_10x10.5" H 5850 1300 50  0001 C CNN
 F 3 "https://eu.mouser.com/datasheet/2/427/517d-239964.pdf" H 5850 1300 50  0001 C CNN
 	1    5850 1300
 	-1   0    0    1
 $EndComp
-Wire Wire Line
-	5250 1050 6750 1050
 Wire Wire Line
 	3600 1050 3600 650
@@
 F 0 "U4" H 4550 3500 50  0000 L BNN
 F 1 "ICL7660SIPAZ" H 4350 2250 50  0000 L BNN
-F 2 "ICL7660SIPAZ:DIP254P762X533-8" H 4550 3000 50  0001 L BNN
-F 3 "Good" H 4550 3000 50  0001 L BNN
+F 2 "Housings_SOIC:SOIC-8_3.9x4.9mm_Pitch1.27mm" H 4550 3000 50  0001 L BNN
+F 3 "https://eu.mouser.com/datasheet/2/698/icl7660-1302119.pdf" H 4550 3000 50  0001 L BNN
 F 4 "ICL7660SIPAZ" H 4550 3000 50  0001 L BNN "Field4"
 F 5 "Intersil" H 4550 3000 50  0001 L BNN "Field5"
@@
 F 0 "C8" H 3625 3150 50  0000 L CNN
 F 1 "10 uF" H 3350 2950 50  0000 L CNN
-F 2 "Capacitors_THT:CP_Radial_D10.0mm_P5.00mm" H 3600 3050 50  0001 C CNN
-F 3 "https://eu.mouser.com/datasheet/2/293/e-upx-876312.pdf" H 3600 3050 50  0001 C CNN
+F 2 "Capacitors_SMD:CP_Elec_4x5.8" H 3600 3050 50  0001 C CNN
+F 3 "https://eu.mouser.com/datasheet/2/315/ABA0000C1251-1138508.pdf" H 3600 3050 50  0001 C CNN
 	1    3600 3050
 	1    0    0    -1
@@
 F 0 "C12" H 5725 2950 50  0000 L CNN
 F 1 "470 uF" H 5725 2750 50  0000 L CNN
-F 2 "Capacitors_THT:CP_Radial_D10.0mm_P5.00mm" H 5700 2850 50  0001 C CNN
+F 2 "Capacitors_SMD:CP_Elec_10x10.5" H 5700 2850 50  0001 C CNN
 F 3 "https://eu.mouser.com/datasheet/2/427/517d-239964.pdf" H 5700 2850 50  0001 C CNN
 	1    5700 2850
@@
 F 0 "U5" H 4550 5150 50  0000 L BNN
 F 1 "ICL7660SIPAZ" H 4350 3900 50  0000 L BNN
-F 2 "ICL7660SIPAZ:DIP254P762X533-8" H 4550 4650 50  0001 L BNN
-F 3 "Good" H 4550 4650 50  0001 L BNN
+F 2 "Housings_SOIC:SOIC-8_3.9x4.9mm_Pitch1.27mm" H 4550 4650 50  0001 L BNN
+F 3 "https://eu.mouser.com/datasheet/2/698/icl7660-1302119.pdf" H 4550 4650 50  0001 L BNN
 F 4 "ICL7660SIPAZ" H 4550 4650 50  0001 L BNN "Field4"
 F 5 "Intersil" H 4550 4650 50  0001 L BNN "Field5"
@@
 F 0 "C9" H 3625 4850 50  0000 L CNN
 F 1 "10 uF" H 3350 4650 50  0000 L CNN
-F 2 "Capacitors_THT:CP_Radial_D10.0mm_P5.00mm" H 3600 4750 50  0001 C CNN
-F 3 "https://eu.mouser.com/datasheet/2/293/e-upx-876312.pdf" H 3600 4750 50  0001 C CNN
+F 2 "Capacitors_SMD:CP_Elec_4x5.8" H 3600 4750 50  0001 C CNN
+F 3 "https://eu.mouser.com/datasheet/2/315/ABA0000C1251-1138508.pdf" H 3600 4750 50  0001 C CNN
 	1    3600 4750
 	1    0    0    -1
@@
 F 0 "C11" H 5675 4550 50  0000 L CNN
 F 1 "470 uF" H 5675 4350 50  0000 L CNN
-F 2 "Capacitors_THT:CP_Radial_D10.0mm_P5.00mm" H 5650 4450 50  0001 C CNN
+F 2 "Capacitors_SMD:CP_Elec_10x10.5" H 5650 4450 50  0001 C CNN
 F 3 "https://eu.mouser.com/datasheet/2/427/517d-239964.pdf" H 5650 4450 50  0001 C CNN
 	1    5650 4450
@@
 Wire Wire Line
 	5250 4250 6700 4250
-Wire Wire Line
-	5400 4550 5400 5550
 Wire Wire Line
 	5400 5550 3300 5550
@@
 F 0 "U6" H 4600 6850 50  0000 L BNN
 F 1 "ICL7660SIPAZ" H 4400 5600 50  0000 L BNN
-F 2 "ICL7660SIPAZ:DIP254P762X533-8" H 4600 6350 50  0001 L BNN
-F 3 "Good" H 4600 6350 50  0001 L BNN
+F 2 "Housings_SOIC:SOIC-8_3.9x4.9mm_Pitch1.27mm" H 4600 6350 50  0001 L BNN
+F 3 "https://eu.mouser.com/datasheet/2/698/icl7660-1302119.pdf" H 4600 6350 50  0001 L BNN
 F 4 "ICL7660SIPAZ" H 4600 6350 50  0001 L BNN "Field4"
 F 5 "Intersil" H 4600 6350 50  0001 L BNN "Field5"
@@
 F 0 "C10" H 3725 6500 50  0000 L CNN
 F 1 "10 uF" H 3450 6300 50  0000 L CNN
-F 2 "Capacitors_THT:CP_Radial_D10.0mm_P5.00mm" H 3700 6400 50  0001 C CNN
-F 3 "https://eu.mouser.com/datasheet/2/293/e-upx-876312.pdf" H 3700 6400 50  0001 C CNN
+F 2 "Capacitors_SMD:CP_Elec_4x5.8" H 3700 6400 50  0001 C CNN
+F 3 "https://eu.mouser.com/datasheet/2/315/ABA0000C1251-1138508.pdf" H 3700 6400 50  0001 C CNN
 	1    3700 6400
 	1    0    0    -1
@@
 F 0 "C13" H 5775 6200 50  0000 L CNN
 F 1 "470 uF" H 5775 6000 50  0000 L CNN
-F 2 "Capacitors_THT:CP_Radial_D10.0mm_P5.00mm" H 5750 6100 50  0001 C CNN
-F 3 "https://eu.mouser.com/datasheet/2/427/517d-239964.pdf" H 5750 6100 50  0001 C CNN
+F 2 "Capacitors_SMD:CP_Elec_10x10.5" H 5750 6100 50  0001 C CNN
+F 3 "https://eu.mouser.com/datasheet/2/315/ABA0000C1145-947633.pdf" H 5750 6100 50  0001 C CNN
 	1    5750 6100
 	-1   0    0    1
 $EndComp
 Wire Wire Line
-	5400 7200 5400 6200
-Wire Wire Line
-	5400 6200 5500 6200
-Wire Wire Line
 	3300 2050 3300 7200
 Wire Wire Line
@@
 	5300 5950 5300 5900
 Wire Wire Line
-	5300 5900 5900 5900
-Text HLabel 6000 5850 2    60   Output ~ 0
+	5300 5900 6000 5900
+Text HLabel 6000 5900 2    60   Output ~ 0
 -8V_3
-Wire Wire Line
-	5900 5900 5900 5850
-Wire Wire Line
-	5900 5850 6000 5850
 Text HLabel 6000 5650 2    60   Output ~ 0
 +8V_3
-Wire Wire Line
-	6000 5650 3300 5650
-Connection ~ 3300 5650
 NoConn ~ 3850 1250
 NoConn ~ 3850 1650
@@
 	3150 5950 3900 5950
 Wire Wire Line
-	5750 1150 5750 1050
-Connection ~ 5750 1050
-Wire Wire Line
 	5550 1450 5850 1450
-Connection ~ 5550 1450
 Wire Wire Line
 	5550 2300 5550 1450
@@
 Wire Wire Line
 	5450 3000 5700 3000
-Connection ~ 5450 3000
 Wire Wire Line
 	5450 3900 5450 3000
 Wire Wire Line
-	5650 5900 5650 5950
-Connection ~ 5650 5900
-Wire Wire Line
-	5500 6250 5750 6250
-Wire Wire Line
-	5500 6200 5500 6250
+	5400 6250 5750 6250
 Wire Wire Line
 	5650 4300 5650 4250
 Connection ~ 5650 4250
 Wire Wire Line
-	5650 4600 5500 4600
-Wire Wire Line
-	5500 4600 5500 4550
-Wire Wire Line
-	5500 4550 5400 4550
+	5400 4600 5650 4600
 Wire Wire Line
 	5650 2700 5700 2700
-Wire Wire Line
-	5850 1150 5750 1150
-Wire Wire Line
-	5650 5950 5750 5950
 Connection ~ 3150 1200
-$Comp
-L PWR_FLAG #FLG04
-U 1 1 5B13D791
-P 2550 1600
-F 0 "#FLG04" H 2550 1675 50  0001 C CNN
-F 1 "PWR_FLAG" H 2550 1750 50  0000 C CNN
-F 2 "" H 2550 1600 50  0001 C CNN
-F 3 "" H 2550 1600 50  0001 C CNN
-	1    2550 1600
-	1    0    0    -1
-$EndComp
-Wire Wire Line
-	2550 1600 2350 1600
-Connection ~ 2350 1600
+Wire Wire Line
+	5400 7200 5400 6250
+Wire Wire Line
+	5400 5550 5400 4600
+Wire Wire Line
+	5750 5950 5750 5900
+Connection ~ 5750 5900
+Wire Wire Line
+	5250 1050 6750 1050
+Wire Wire Line
+	5850 1150 5850 1050
+Connection ~ 5850 1050
+Wire Wire Line
+	6000 5650 3150 5650
+Connection ~ 3150 5650
+Wire Wire Line
+	3700 2300 3700 2050
+Connection ~ 3700 2050
 $EndSCHEMATC

Commit message: Shis ir mans meeginaajums iztraseet plati ( nepabeigts- vajag paliidziibu)
Parts:
- added J21, J22, J23, J24, J25, J26, J27, J28, J29, J30, J31, J32, J33, J37: Conn_01x01, Measurement_Points:Measurement_Point_Round-TH_Small, symbol Conn_01x01
Connections:
- net +8V: now also J21.1 (Pin_1), J22.1 (Pin_1), J23.1 (Pin_1), J24.1 (Pin_1), J25.1 (Pin_1)
- net -8V: now also J26.1 (Pin_1), J27.1 (Pin_1)
- net -8V_1: now also J28.1 (Pin_1), J29.1 (Pin_1)
- net -8V_2: now also J30.1 (Pin_1), J31.1 (Pin_1), J37.1 (Pin_1)
- net -8V_3: now also J32.1 (Pin_1), J33.1 (Pin_1)

Commit message: Kursa/Prakses darba pabeigtaa plates versija
Parts:
- added J38, J47, J48, J49, J50, J51: Conn_01x01, Measurement_Points:Measurement_Point_Round-TH_Small, symbol Conn_01x01
Connections:
- net +8V: now also J47.1 (Pin_1), J48.1 (Pin_1), J49.1 (Pin_1), J51.1 (Pin_1)
- net -8V: now also J50.1 (Pin_1)
- net -8V_1: now also J38.1 (Pin_1)
Changed lines of the file:
@@
 	8300 3350 8300 3450
 Connection ~ 8300 3450
+$Comp
+L Conn_01x01 J38
+U 1 1 5B203C5E
+P 7500 3050
+F 0 "J38" H 7500 3150 50  0000 C CNN
+F 1 "Conn_01x01" H 7500 2950 50  0000 C CNN
+F 2 "Measurement_Points:Measurement_Point_Round-TH_Small" H 7500 3050 50  0001 C CNN
+F 3 "" H 7500 3050 50  0001 C CNN
+	1    7500 3050
+	0    1    1    0
+$EndComp
+Wire Wire Line
+	7500 2800 7500 2850
+Connection ~ 7500 2800
+$Comp
+L Conn_01x01 J47
+U 1 1 5B2115C6
+P 8300 1200
+F 0 "J47" H 8300 1300 50  0000 C CNN
+F 1 "Conn_01x01" H 8300 1100 50  0000 C CNN
+F 2 "Measurement_Points:Measurement_Point_Round-TH_Small" H 8300 1200 50  0001 C CNN
+F 3 "" H 8300 1200 50  0001 C CNN
+	1    8300 1200
+	-1   0    0    1
+$EndComp
+$Comp
+L Conn_01x01 J48
+U 1 1 5B211659
+P 8300 1500
+F 0 "J48" H 8300 1600 50  0000 C CNN
+F 1 "Conn_01x01" H 8300 1400 50  0000 C CNN
+F 2 "Measurement_Points:Measurement_Point_Round-TH_Small" H 8300 1500 50  0001 C CNN
+F 3 "" H 8300 1500 50  0001 C CNN
+	1    8300 1500
+	-1   0    0    1
+$EndComp
+$Comp
+L Conn_01x01 J49
+U 1 1 5B2116F3
+P 8300 1850
+F 0 "J49" H 8300 1950 50  0000 C CNN
+F 1 "Conn_01x01" H 8300 1750 50  0000 C CNN
+F 2 "Measurement_Points:Measurement_Point_Round-TH_Small" H 8300 1850 50  0001 C CNN
+F 3 "" H 8300 1850 50  0001 C CNN
+	1    8300 1850
+	-1   0    0    1
+$EndComp
+Wire Wire Line
+	8450 850  8700 850
+Connection ~ 8700 850
+Wire Wire Line
+	8500 1200 8700 1200
+Connection ~ 8700 1200
+$Comp
+L Conn_01x01 J50
+U 1 1 5B211B78
+P 8450 2450
+F 0 "J50" H 8450 2550 50  0000 C CNN
+F 1 "Conn_01x01" H 8450 2350 50  0000 C CNN
+F 2 "Measurement_Points:Measurement_Point_Round-TH_Small" H 8450 2450 50  0001 C CNN
+F 3 "" H 8450 2450 50  0001 C CNN
+	1    8450 2450
+	-1   0    0    1
+$EndComp
+Wire Wire Line
+	8750 2450 8650 2450
+Connection ~ 8750 2450
+$Comp
+L Conn_01x01 J51
+U 1 1 5B20E1AA
+P 8250 850
+F 0 "J51" H 8250 950 50  0000 C CNN
+F 1 "Conn_01x01" H 8250 750 50  0000 C CNN
+F 2 "Measurement_Points:Measurement_Point_Round-TH_Small" H 8250 850 50  0001 C CNN
+F 3 "" H 8250 850 50  0001 C CNN
+	1    8250 850
+	-1   0    0    1
+$EndComp
+Wire Wire Line
+	8500 1850 8700 1850
+Connection ~ 8700 1850
+Wire Wire Line
+	8700 1500 8500 1500
+Connection ~ 8700 1500
 $EndSCHEMATC

Commit message: 1. Prototipa finaala versija
Parts:
- added J100, J101, J102, J103, J104, J105, J106, J107, J108, J109, J110, J111, J112, J113, J114, J53, J68, J69, J70, J71, J72, J73, J74, J75, J76, J77, J78, J79, J80, J81, J82, J83, J84, J85, J86, J87, J88, J89, J90, J91, J92, J93, J94, J95, J96, J97, J98, J99: Conn_01x01, Measurement_Points:Measurement_Point_Round-TH_Small, symbol Conn_01x01
Connections:
- net +12V: now also J53.1 (Pin_1)
- net GND: now also U5.3 (GND), J100.1 (Pin_1), J101.1 (Pin_1), J102.1 (Pin_1), J103.1 (Pin_1), J104.1 (Pin_1), J105.1 (Pin_1), J106.1 (Pin_1), J107.1 (Pin_1), J108.1 (Pin_1), J109.1 (Pin_1), J110.1 (Pin_1), J111.1 (Pin_1), J112.1 (Pin_1), J113.1 (Pin_1), J114.1 (Pin_1), J68.1 (Pin_1), J69.1 (Pin_1), J70.1 (Pin_1), J71.1 (Pin_1), J72.1 (Pin_1), J73.1 (Pin_1), J74.1 (Pin_1), J75.1 (Pin_1), J76.1 (Pin_1), J77.1 (Pin_1), J78.1 (Pin_1), J79.1 (Pin_1), J80.1 (Pin_1), J81.1 (Pin_1), J82.1 (Pin_1), J83.1 (Pin_1), J84.1 (Pin_1), J85.1 (Pin_1), J86.1 (Pin_1), J87.1 (Pin_1), J88.1 (Pin_1), J89.1 (Pin_1), J90.1 (Pin_1), J91.1 (Pin_1), J92.1 (Pin_1), J93.1 (Pin_1), J94.1 (Pin_1), J95.1 (Pin_1), J96.1 (Pin_1), J97.1 (Pin_1), J98.1 (Pin_1), J99.1 (Pin_1)
- no-connect marks 13 -> 12
