File: Kursa_darbs_Klavs_Ozols/Kursa_darbs_Klavs_Ozols.sch (KiCad schematic (older format))
At the start: 2 parts, among them J1 Barosana, J2 Audio-Jack-2

Commit message: Shii ir kursa darba 3. iteraacija
Parts:
- removed J2: Audio-Jack-2, symbol Audio-Jack-2
- added J2: Audio-Jack-3, Audio_Jack:Audio_Jack_3.5_mm_Stereo, symbol Audio-Jack-3
- J1: footprint (none) -> Connectors:BARREL_JACK
Changed lines of the file:
@@
 F 0 "J1" H 800 1650 50  0000 C CNN
 F 1 "Barosana" H 800 1350 50  0000 C CNN
-F 2 "" H 800 1550 50  0001 C CNN
-F 3 "" H 800 1550 50  0001 C CNN
+F 2 "Connectors:BARREL_JACK" H 800 1550 50  0001 C CNN
+F 3 "https://eu.mouser.com/datasheet/2/222/STX3200-334669.pdf" H 800 1550 50  0001 C CNN
 	1    800  1550
 	-1   0    0    1
@@
 Wire Wire Line
 	1750 5250 3700 5250
+Entry Wire Line
+	3950 5000 4050 5100
+Wire Wire Line
+	3950 5000 3700 5000
+Wire Wire Line
+	3700 5000 3700 5250
+Text Label 3700 5000 0    60   ~ 0
+Audio
 $Comp
-L Audio-Jack-2 J2
-U 1 1 5B042999
-P 1600 5400
-F 0 "J2" H 1575 5475 50  0000 C CNN
-F 1 "Audio-Jack-2" H 1575 5225 50  0000 C CNN
-F 2 "" H 1850 5400 50  0001 C CNN
-F 3 "" H 1850 5400 50  0001 C CNN
-	1    1600 5400
+L Audio-Jack-3 J2
+U 1 1 5B0C7932
+P 1550 5150
+F 0 "J2" H 1500 5325 50  0000 C CNN
+F 1 "Audio-Jack-3" H 1650 5000 50  0000 C CNN
+F 2 "Audio_Jack:Audio_Jack_3.5_mm_Stereo" H 1800 5250 50  0001 C CNN
+F 3 "https://eu.mouser.com/datasheet/2/222/STX3120-334667.pdf" H 1800 5250 50  0001 C CNN
+	1    1550 5150
 	1    0    0    -1
 $EndComp
 Wire Wire Line
-	1800 5500 1800 5700
-Wire Wire Line
-	1800 5700 1350 5700
-Wire Wire Line
-	1350 5700 1350 5450
-Wire Wire Line
-	1750 5250 1750 5350
-Wire Wire Line
-	1750 5350 1800 5350
-Wire Wire Line
-	1800 5350 1800 5400
-Entry Wire Line
-	3950 5000 4050 5100
-Wire Wire Line
-	3950 5000 3700 5000
-Wire Wire Line
-	3700 5000 3700 5250
-Text Label 3700 5000 0    60   ~ 0
-Audio
+	1350 5450 1350 5250
+Wire Wire Line
+	1750 5050 1800 5050
+Wire Wire Line
+	1800 5050 1800 5200
+Wire Wire Line
+	1800 5200 1750 5200
+Wire Wire Line
+	1750 5200 1750 5250
+Wire Wire Line
+	1750 5150 1800 5150
+Connection ~ 1800 5150
 $EndSCHEMATC

Commit message: Shiii ir 5. iteraacija manai platei - layouts
Parts:
- added J3, J4, J5, J6, J7, J8: Conn_01x01, Mounting_Holes:MountingHole_3.2mm_M3_Pad_Via, symbol Conn_01x01
Connections:
- net GND: now also J3.1 (Pin_1), J4.1 (Pin_1), J5.1 (Pin_1), J6.1 (Pin_1), J7.1 (Pin_1), J8.1 (Pin_1)
Changed lines of the file:
@@
 EESchema Schematic File Version 2
+LIBS:Kursa_darbs_Klavs_Ozols-rescue
 LIBS:power
 LIBS:device
@@
 F20 "Audio10kHz" I L 7650 2500 60
 F21 "Audio10kHz-R" O R 10000 2350 60
-F22 "Audio25Hz" I L 7650 2650 60
-F23 "Audio25kHz-R" O R 10000 2600 60
-F24 "-8V_2" I L 7650 850 60
+F22 "Audio25kHz-R" O R 10000 2600 60
+F23 "-8V_2" I L 7650 850 60
+F24 "Audio25kHz" I L 7650 2650 60
 $EndSheet
 Entry Wire Line
@@
 Wire Wire Line
 	900  1300 900  1250
-Wire Wire Line
-	1350 5450 1150 5450
-Wire Wire Line
-	1150 5450 1150 2650
 Connection ~ 1400 2650
-Wire Wire Line
-	1750 5250 3700 5250
-Entry Wire Line
-	3950 5000 4050 5100
-Wire Wire Line
-	3950 5000 3700 5000
-Wire Wire Line
-	3700 5000 3700 5250
-Text Label 3700 5000 0    60   ~ 0
+Entry Wire Line
+	3950 5150 4050 5250
+Text Label 3700 5150 0    60   ~ 0
 Audio
 $Comp
@@
 $EndComp
 Wire Wire Line
-	1350 5450 1350 5250
-Wire Wire Line
-	1750 5050 1800 5050
-Wire Wire Line
-	1800 5050 1800 5200
-Wire Wire Line
-	1800 5200 1750 5200
-Wire Wire Line
-	1750 5200 1750 5250
-Wire Wire Line
-	1750 5150 1800 5150
-Connection ~ 1800 5150
+	1750 5050 1850 5050
+Wire Wire Line
+	1850 5150 1750 5150
+Wire Wire Line
+	1850 5100 3700 5100
+Wire Wire Line
+	1850 5050 1850 5150
+Connection ~ 1850 5100
+Wire Wire Line
+	3950 5150 3700 5150
+Wire Wire Line
+	3700 5150 3700 5100
+Wire Wire Line
+	1150 2650 1150 5250
+Wire Wire Line
+	1150 5250 1350 5250
+$Comp
+L PWR_FLAG #FLG04
+U 1 1 5B160CE3
+P 850 1750
+F 0 "#FLG04" H 850 1825 50  0001 C CNN
+F 1 "PWR_FLAG" H 850 1900 50  0000 C CNN
+F 2 "" H 850 1750 50  0001 C CNN
+F 3 "" H 850 1750 50  0001 C CNN
+	1    850  1750
+	-1   0    0    1
+$EndComp
+Wire Wire Line
+	1100 1600 950  1600
+Wire Wire Line
+	950  1600 950  1750
+Wire Wire Line
+	950  1750 850  1750
+Connection ~ 1100 1600
+$Comp
+L Conn_01x01 J3
+U 1 1 5B1CA91A
+P 1050 2150
+F 0 "J3" H 1200 2200 50  0000 C CNN
+F 1 "Conn_01x01" H 1350 2100 50  0000 C CNN
+F 2 "Mounting_Holes:MountingHole_3.2mm_M3_Pad_Via" H 1050 2150 50  0001 C CNN
+F 3 "" H 1050 2150 50  0001 C CNN
+	1    1050 2150
+	-1   0    0    1
+$EndComp
+$Comp
+L Conn_01x01 J4
+U 1 1 5B1CAB95
+P 1050 2350
+F 0 "J4" H 1050 2450 50  0000 C CNN
+F 1 "Conn_01x01" H 1350 2300 50  0000 C CNN
+F 2 "Mounting_Holes:MountingHole_3.2mm_M3_Pad_Via" H 1050 2350 50  0001 C CNN
+F 3 "" H 1050 2350 50  0001 C CNN
+	1    1050 2350
+	-1   0    0    1
+$EndComp
+$Comp
+L Conn_01x01 J5
+U 1 1 5B1CADCF
+P 1050 2550
+F 0 "J5" H 1150 2600 50  0000 C CNN
+F 1 "Conn_01x01" H 1350 2500 50  0000 C CNN
+F 2 "Mounting_Holes:MountingHole_3.2mm_M3_Pad_Via" H 1050 2550 50  0001 C CNN
+F 3 "" H 1050 2550 50  0001 C CNN
+	1    1050 2550
+	-1   0    0    1
+$EndComp
+$Comp
+L Conn_01x01 J6
+U 1 1 5B1CB33C
+P 850 2850
+F 0 "J6" H 850 2950 50  0000 C CNN
+F 1 "Conn_01x01" H 950 2750 50  0000 C CNN
+F 2 "Mounting_Holes:MountingHole_3.2mm_M3_Pad_Via" H 850 2850 50  0001 C CNN
+F 3 "" H 850 2850 50  0001 C CNN
+	1    850  2850
+	-1   0    0    1
+$EndComp
+Wire Wire Line
+	1400 2550 1250 2550
+Connection ~ 1400 2550
+Wire Wire Line
+	1400 2350 1250 2350
+Connection ~ 1400 2350
+Wire Wire Line
+	1400 2150 1250 2150
+Connection ~ 1400 2150
+Wire Wire Line
+	1150 2850 1050 2850
+Connection ~ 1150 2850
+$Comp
+L Conn_01x01 J7
+U 1 1 5B1CEB89
+P 850 3150
+F 0 "J7" H 850 3250 50  0000 C CNN
+F 1 "Conn_01x01" H 950 3050 50  0000 C CNN
+F 2 "Mounting_Holes:MountingHole_3.2mm_M3_Pad_Via" H 850 3150 50  0001 C CNN
+F 3 "" H 850 3150 50  0001 C CNN
+	1    850  3150
+	-1   0    0    1
+$EndComp
+$Comp
+L Conn_01x01 J8
+U 1 1 5B1CEDD8
+P 850 3450
+F 0 "J8" H 850 3550 50  0000 C CNN
+F 1 "Conn_01x01" H 950 3350 50  0000 C CNN
+F 2 "Mounting_Holes:MountingHole_3.2mm_M3_Pad_Via" H 850 3450 50  0001 C CNN
+F 3 "" H 850 3450 50  0001 C CNN
+	1    850  3450
+	-1   0    0    1
+$EndComp
+Wire Wire Line
+	1050 3150 1150 3150
+Connection ~ 1150 3150
+Wire Wire Line
+	1050 3450 1150 3450
+Connection ~ 1150 3450
 $EndSCHEMATC

Commit message: Shis ir mans meeginaajums iztraseet plati ( nepabeigts- vajag paliidziibu)
Parts:
- added J11, J12, J13, J14, J15, J16, J17, J18, J19, J20, J34, J35, J36, J9: Conn_01x01, Measurement_Points:Measurement_Point_Round-TH_Small, symbol Conn_01x01
Connections:
- net +12V: now also J9.1 (Pin_1)
- net 10k: now also J14.1 (Pin_1)
- net 1k: now also J13.1 (Pin_1)
- net 200: now also J12.1 (Pin_1)
- net 25 kHz - 470 pF/Audio25kHz: now also J35.1 (Pin_1), J36.1 (Pin_1)
- net 50: now also J11.1 (Pin_1)
- net Audio: now also J15.1 (Pin_1), J16.1 (Pin_1), J17.1 (Pin_1)
- net GND: now also J18.1 (Pin_1), J19.1 (Pin_1), J20.1 (Pin_1), J34.1 (Pin_1)

Commit message: Kursa/Prakses darba pabeigtaa plates versija
Parts:
- added J39, J40, J41, J42, J43, J44, J45, J46, J52: Conn_01x01, Measurement_Points:Measurement_Point_Round-TH_Small, symbol Conn_01x01
Connections:
- net 10: now also J52.1 (Pin_1)
- net 10 kHz - 1 nF/Audio10kHz: now also J45.1 (Pin_1), J46.1 (Pin_1)
- net 10Hz-100nF/Audio10Hz: now also J11.1 (Pin_1), J12.1 (Pin_1)
- net 10k: no longer J14.1 (Pin_1)
- net 1k: no longer J13.1 (Pin_1)
- net 1kHz -10 nF/Audio1kHz: now also J39.1 (Pin_1), J40.1 (Pin_1)
- net 2.5 kHz- 4.7 nF/Audio2.5kHz: now also J41.1 (Pin_1), J42.1 (Pin_1)
- net 200: no longer J12.1 (Pin_1)
- net 200Hz - 47nF/Audio200Hz: now also J18.1 (Pin_1), J19.1 (Pin_1)
- net 4.5kHz - 2.2 nF/Audio4.5kHz: now also J43.1 (Pin_1), J44.1 (Pin_1)
- net 50: no longer J11.1 (Pin_1)
- net 500Hz - 22 nF/Audio500Hz: now also J20.1 (Pin_1), J34.1 (Pin_1)
- net 50Hz - 220 nF/Audio50Hz: now also J13.1 (Pin_1), J14.1 (Pin_1)
- net GND: no longer J18.1 (Pin_1), J19.1 (Pin_1), J20.1 (Pin_1), J34.1 (Pin_1)

Commit message: 1. Prototipa finaala versija
Parts:
- added J54, J55, J56, J57, J58, J59, J60, J61, J62, J63, J64, J65, J66, J67: Conn_01x01, Mounting_Holes:MountingHole_3.2mm_M3_Pad_Via, symbol Conn_01x01
Connections:
- net GND: now also J54.1 (Pin_1), J55.1 (Pin_1), J56.1 (Pin_1), J57.1 (Pin_1), J58.1 (Pin_1), J59.1 (Pin_1), J60.1 (Pin_1), J61.1 (Pin_1), J62.1 (Pin_1), J63.1 (Pin_1), J64.1 (Pin_1), J65.1 (Pin_1), J66.1 (Pin_1), J67.1 (Pin_1)
Changed lines of the file:
@@
 	10150 700  10150 950
 Connection ~ 10150 950
+$Comp
+L Conn_01x01 J57
+U 1 1 5B255C18
+P 850 3750
+F 0 "J57" H 850 3850 50  0000 C CNN
+F 1 "Conn_01x01" H 950 3650 50  0000 C CNN
+F 2 "Mounting_Holes:MountingHole_3.2mm_M3_Pad_Via" H 850 3750 50  0001 C CNN
+F 3 "" H 850 3750 50  0001 C CNN
+	1    850  3750
+	-1   0    0    1
+$EndComp
+$Comp
+L Conn_01x01 J59
+U 1 1 5B256229
+P 850 4000
+F 0 "J59" H 850 4100 50  0000 C CNN
+F 1 "Conn_01x01" H 950 3900 50  0000 C CNN
+F 2 "Mounting_Holes:MountingHole_3.2mm_M3_Pad_Via" H 850 4000 50  0001 C CNN
+F 3 "" H 850 4000 50  0001 C CNN
+	1    850  4000
+	-1   0    0    1
+$EndComp
+$Comp
+L Conn_01x01 J61
+U 1 1 5B2564BA
+P 850 4250
+F 0 "J61" H 850 4350 50  0000 C CNN
+F 1 "Conn_01x01" H 950 4150 50  0000 C CNN
+F 2 "Mounting_Holes:MountingHole_3.2mm_M3_Pad_Via" H 850 4250 50  0001 C CNN
+F 3 "" H 850 4250 50  0001 C CNN
+	1    850  4250
+	-1   0    0    1
+$EndComp
+$Comp
+L Conn_01x01 J63
+U 1 1 5B2569A6
+P 850 4550
+F 0 "J63" H 850 4650 50  0000 C CNN
+F 1 "Conn_01x01" H 950 4450 50  0000 C CNN
+F 2 "Mounting_Holes:MountingHole_3.2mm_M3_Pad_Via" H 850 4550 50  0001 C CNN
+F 3 "" H 850 4550 50  0001 C CNN
+	1    850  4550
+	-1   0    0    1
+$EndComp
+$Comp
+L Conn_01x01 J65
+U 1 1 5B256C3D
+P 850 4800
+F 0 "J65" H 850 4900 50  0000 C CNN
+F 1 "Conn_01x01" H 950 4700 50  0000 C CNN
+F 2 "Mounting_Holes:MountingHole_3.2mm_M3_Pad_Via" H 850 4800 50  0001 C CNN
+F 3 "" H 850 4800 50  0001 C CNN
+	1    850  4800
+	-1   0    0    1
+$EndComp
+$Comp
+L Conn_01x01 J66
+U 1 1 5B256ED9
+P 850 5050
+F 0 "J66" H 850 5150 50  0000 C CNN
+F 1 "Conn_01x01" H 950 4950 50  0000 C CNN
+F 2 "Mounting_Holes:MountingHole_3.2mm_M3_Pad_Via" H 850 5050 50  0001 C CNN
+F 3 "" H 850 5050 50  0001 C CNN
+	1    850  5050
+	-1   0    0    1
+$EndComp
+$Comp
+L Conn_01x01 J67
+U 1 1 5B257178
+P 850 5350
+F 0 "J67" H 850 5450 50  0000 C CNN
+F 1 "Conn_01x01" H 950 5250 50  0000 C CNN
+F 2 "Mounting_Holes:MountingHole_3.2mm_M3_Pad_Via" H 850 5350 50  0001 C CNN
+F 3 "" H 850 5350 50  0001 C CNN
+	1    850  5350
+	-1   0    0    1
+$EndComp
+$Comp
+L Conn_01x01 J54
+U 1 1 5B257549
+P 1450 2950
+F 0 "J54" H 1450 3050 50  0000 C CNN
+F 1 "Conn_01x01" H 1550 2850 50  0000 C CNN
+F 2 "Mounting_Holes:MountingHole_3.2mm_M3_Pad_Via" H 1450 2950 50  0001 C CNN
+F 3 "" H 1450 2950 50  0001 C CNN
+	1    1450 2950
+	1    0    0    -1
+$EndComp
+$Comp
+L Conn_01x01 J55
+U 1 1 5B257A84
+P 1450 3250
+F 0 "J55" H 1450 3350 50  0000 C CNN
+F 1 "Conn_01x01" H 1550 3150 50  0000 C CNN
+F 2 "Mounting_Holes:MountingHole_3.2mm_M3_Pad_Via" H 1450 3250 50  0001 C CNN
+F 3 "" H 1450 3250 50  0001 C CNN
+	1    1450 3250
+	1    0    0    -1
+$EndComp
+$Comp
+L Conn_01x01 J56
+U 1 1 5B257D34
+P 1450 3550
+F 0 "J56" H 1450 3650 50  0000 C CNN
+F 1 "Conn_01x01" H 1550 3450 50  0000 C CNN
+F 2 "Mounting_Holes:MountingHole_3.2mm_M3_Pad_Via" H 1450 3550 50  0001 C CNN
+F 3 "" H 1450 3550 50  0001 C CNN
+	1    1450 3550
+	1    0    0    -1
+$EndComp
+$Comp
+L Conn_01x01 J58
+U 1 1 5B257FDD
+P 1450 3850
+F 0 "J58" H 1450 3950 50  0000 C CNN
+F 1 "Conn_01x01" H 1550 3750 50  0000 C CNN
+F 2 "Mounting_Holes:MountingHole_3.2mm_M3_Pad_Via" H 1450 3850 50  0001 C CNN
+F 3 "" H 1450 3850 50  0001 C CNN
+	1    1450 3850
+	1    0    0    -1
+$EndComp
+$Comp
+L Conn_01x01 J60
+U 1 1 5B2589FD
+P 1450 4150
+F 0 "J60" H 1450 4250 50  0000 C CNN
+F 1 "Conn_01x01" H 1550 4050 50  0000 C CNN
+F 2 "Mounting_Holes:MountingHole_3.2mm_M3_Pad_Via" H 1450 4150 50  0001 C CNN
+F 3 "" H 1450 4150 50  0001 C CNN
+	1    1450 4150
+	1    0    0    -1
+$EndComp
+$Comp
+L Conn_01x01 J62
+U 1 1 5B258CBA
+P 1450 4450
+F 0 "J62" H 1450 4550 50  0000 C CNN
+F 1 "Conn_01x01" H 1550 4350 50  0000 C CNN
+F 2 "Mounting_Holes:MountingHole_3.2mm_M3_Pad_Via" H 1450 4450 50  0001 C CNN
+F 3 "" H 1450 4450 50  0001 C CNN
+	1    1450 4450
+	1    0    0    -1
+$EndComp
+$Comp
+L Conn_01x01 J64
+U 1 1 5B258F6C
+P 1450 4750
+F 0 "J64" H 1450 4850 50  0000 C CNN
+F 1 "Conn_01x01" H 1550 4650 50  0000 C CNN
+F 2 "Mounting_Holes:MountingHole_3.2mm_M3_Pad_Via" H 1450 4750 50  0001 C CNN
+F 3 "" H 1450 4750 50  0001 C CNN
+	1    1450 4750
+	1    0    0    -1
+$EndComp
+Wire Wire Line
+	1250 2950 1150 2950
+Connection ~ 1150 2950
+Wire Wire Line
+	1250 3250 1150 3250
+Connection ~ 1150 3250
+Wire Wire Line
+	1250 3550 1150 3550
+Connection ~ 1150 3550
+Wire Wire Line
+	1050 3750 1150 3750
+Connection ~ 1150 3750
+Wire Wire Line
+	1250 3850 1150 3850
+Connection ~ 1150 3850
+Wire Wire Line
+	1050 4000 1150 4000
+Connection ~ 1150 4000
+Wire Wire Line
+	1250 4150 1150 4150
+Connection ~ 1150 4150
+Wire Wire Line
+	1050 4250 1150 4250
+Connection ~ 1150 4250
+Wire Wire Line
+	1250 4450 1150 4450
+Connection ~ 1150 4450
+Wire Wire Line
+	1050 4550 1150 4550
+Connection ~ 1150 4550
+Wire Wire Line
+	1250 4750 1150 4750
+Connection ~ 1150 4750
+Wire Wire Line
+	1050 4800 1150 4800
+Connection ~ 1150 4800
+Wire Wire Line
+	1050 5050 1150 5050
+Connection ~ 1150 5050
+Wire Wire Line
+	1050 5350 1200 5350
+Wire Wire Line
+	1200 5350 1200 5250
+Connection ~ 1200 5250
 $EndSCHEMATC
